Commit message: Moved to the updated husky package.

File: husky/husky_description/urdf/accessories/kinect_camera.urdf.xacro (robot description, xacro)
@@ -38,4 +38,5 @@
       </visual>
       <collision>
+	<origin xyz="0 0 0" rpy="0 0 ${M_PI/2}"/>
         <geometry>
           <box size="0.07 0.3 0.09"/>

File: husky/husky_description/urdf/accessories/sensor_arch.urdf.xacro (robot description, xacro)
@@ -13,5 +13,5 @@
                  <origin xyz="0 0 0" rpy="0 0 0"/>
                  <geometry>
-                     <mesh filename="package://husky_description/meshes/accessories/${size}_mm_sensor_arch.dae" />
+                     <mesh filename="package://husky_description/meshes/accessories/${size}_mm_sensor_arch.stl" />
                  </geometry>
              </collision>

File: husky/husky_description/urdf/accessories/sick_lms1xx_mount.urdf.xacro (robot description, xacro)
@@ -31,5 +31,5 @@
     <link name="${prefix}_laser_mount">
       <visual>
-        <origin xyz="0 0 0" rpy="0 0 ${-M_PI/2}" />
+        <origin xyz="0 0 0" rpy="0 ${-M_PI} ${-M_PI/2}" />
         <geometry>
           <!-- Origin of this mesh is the base of the bracket. -->
@@ -38,5 +38,5 @@
       </visual>
       <collision>
-        <origin xyz="0 0 .0585" rpy="0 0 0" />
+        <origin xyz="0 0 .0585" rpy="0 ${-M_PI} ${-M_PI/2}" />
         <geometry>
           <box size=".1 .108 .117" />
@@ -46,5 +46,5 @@
     <joint name="${prefix}_laser_joint" type="fixed">
       <!-- This offset is from the base of the bracket to the LIDAR's focal point. -->
-      <origin xyz="0.0352 0 0.0566" rpy="${M_PI} 0 0" />
+      <origin xyz="-0.0352 0 -0.0566" rpy="0 0 0" />
       <parent link="${prefix}_laser_mount" />
       <child link="${prefix}_laser" />

File: husky/husky_description/urdf/decorations.urdf.xacro (robot description, xacro)
@@ -51,5 +51,5 @@
       <child link="user_rail_link" />
     </joint>
-    <!-- Spawn front bumper link -->
+    <!-- Spawn front bumper link
     <link name="front_bumper_link">
       <visual>
@@ -58,11 +58,11 @@
         </geometry>
       </visual>
-    </link>
-    <!-- Attach front bumper -->
+    </link> -->
+    <!-- Attach front bumper
     <joint name="front_bumper" type="fixed">
       <origin xyz="0.48 0 0.091" rpy="0 0 0" />
       <parent link="base_link" />
       <child link="front_bumper_link" />
-    </joint>
+    </joint> -->
     <!-- Spawn rear bumper link -->
     <link name="rear_bumper_link">
@@ -91,5 +91,5 @@
           <origin xyz="0 0 0" rpy="0 0 0"/>
           <geometry>
-            <mesh filename="package://husky_description/meshes/top_plate.dae" />
+            <mesh filename="package://husky_description/meshes/top_plate.stl" />
           </geometry>
         </collision>

File: husky/husky_description/urdf/description.xacro (robot description, xacro)
@@ -24,5 +24,8 @@
   <xacro:arg name="laser_enabled" default="false" />
   <xacro:arg name="ur5_enabled" default="false" />
+  <xacro:arg name="ur5_camera_enabled" default="false" />
   <xacro:arg name="kinect_enabled" default="false" />
+  <xacro:arg name="kinectv2_enabled" default="false" />
+  <xacro:arg name="primesense_enabled" default="false"/>
   <xacro:include filename="$(find husky_description)/urdf/husky.urdf.xacro" />
   <xacro:husky_robot />

File: husky/husky_description/urdf/husky.urdf.xacro (robot description, xacro)
@@ -26,4 +26,6 @@
   <xacro:include filename="$(find husky_description)/urdf/wheel.urdf.xacro" />
   <xacro:include filename="$(find husky_description)/urdf/accessories/kinect_camera.urdf.xacro"/>
+  <xacro:include filename="$(find husky_description)/urdf/accessories/kinectv2_camera.urdf.xacro"/>
+  <xacro:include filename="$(find husky_description)/urdf/accessories/primesense_carmine_1-09_camera.urdf.xacro"/>
   <xacro:include filename="$(find husky_description)/urdf/accessories/sick_lms1xx_mount.urdf.xacro"/>
   <xacro:include filename="$(find husky_description)/urdf/accessories/sensor_arch.urdf.xacro"/>
@@ -74,7 +76,7 @@
     <link name="inertial_link">
       <inertial>
-        <mass value="330.455" />
+        <mass value="80" />
         <origin xyz="-0.08748 -0.00085 0.09947" />
-        <inertia ixx="10.6022" ixy="-0.02364" ixz="-0.1197" iyy="10.7386" iyz="-0.001544" izz="20.0296" />
+        <inertia ixx="1.08995475113" ixy="-0.0427873303" ixz="-0.2166515837" iyy="3.14678733031" iyz="-0.00279457012" izz="3.67348416289" />
       </inertial>
     </link>
@@ -88,5 +90,5 @@
     <link name="imu_link"/>
     <joint name="imu_joint" type="fixed">
-      <origin xyz="$(optenv HUSKY_IMU_XYZ 0.19 0 0.149)" rpy="$(optenv HUSKY_IMU_RPY 0 -1.5708 3.1416)" />
+      <origin xyz="$(optenv HUSKY_IMU_XYZ 0.19 0 0.149)" rpy="$(optenv HUSKY_IMU_RPY 0 -1.57079632679 3.14159265359)" />
       <parent link="base_link" />
       <child link="imu_link" />
@@ -116,5 +118,5 @@
         <parent link="top_plate_link" />
         <child link="ur5_arm_base_link" />
-        <origin xyz="0.3058 0 0.0065" rpy="0.0 0.0 -1.57" />
+        <origin xyz="0.3058 0 0.0065" rpy="0.0 0.0 -1.57079632679" />
       </joint>
       <!-- Spawn gripper-->
@@ -127,8 +129,20 @@
         </joint>
     </xacro:if>
+    <xacro:if value="$(arg ur5_camera_enabled)">
+      <xacro:property name="reflect" value="-1" />
+      <!-- Spawn arm -->
+      <xacro:ur5_robot prefix="ur5_arm_" joint_limited="true"/>
+      <!-- Join arm -->
+      <joint name="ur5_arm_base" type="fixed">
+        <parent link="top_plate_link" />
+        <child link="ur5_arm_base_link" />
+        <origin xyz="0.3058 0 0.0065" rpy="0.0 0.0 -1.57079632679" />
+      </joint>
+    </xacro:if>
+    <!-- Spawn LIDAR if laser_enabled = "true" -->
     <xacro:if value="$(arg laser_enabled)">
       <sick_lms1xx_mount prefix="base" topic="scan"/>
       <joint name="laser_mount_joint" type="fixed">
-        <origin xyz="$(optenv HUSKY_LMS1XX_XYZ 0.415 0.0 -0.14)"
+        <origin xyz="$(optenv HUSKY_LMS1XX_XYZ 0.415 0.0 -0.04)"
                 rpy="$(optenv HUSKY_LMS1XX_RPY 0.0 0.0 0.0)" />
         <parent link="top_plate_link" />
@@ -136,14 +150,99 @@
       </joint>
     </xacro:if>
+    <!-- Spawn Kinect if kinect_enabled = "true" -->
     <xacro:if value="$(arg kinect_enabled)">
       <xacro:sensor_arch prefix="" parent="top_plate_link">
-        <origin xyz="-0.35 0 0.51" rpy="0 0 -3.14"/>
+        <origin xyz="-0.35 0 0.51" rpy="0 0 -3.14159265359"/>
       </xacro:sensor_arch>
       <joint name="kinect_frame_joint" type="fixed">
-        <origin xyz="$(optenv HUSKY_KINECT_XYZ 0 0 0)" rpy="$(optenv HUSKY_KINECT_RPY 0 0.18 3.14)" />
+        <origin xyz="$(optenv HUSKY_KINECT_XYZ 0 0 0)" rpy="$(optenv HUSKY_KINECT_RPY 0 0.18 3.14159265359)" />
         <parent link="sensor_arch_mount_link"/>
         <child link="camera_link"/>
       </joint>
       <xacro:kinect_camera prefix="camera"/>
+      <link name="camera_optical_frame"/>
+      <joint name="camera_optical_joint" type="fixed">
+        <origin xyz="0 0 0" rpy="-1.57079632679 0 -1.57079632679"/>
+        <parent link="camera_link"/>
+        <child link="camera_optical_frame"/>
+      </joint>
+    </xacro:if>
+    <!-- Spawn KinectV2 if kinectv2_enabled = "true" -->
+    <xacro:if value="$(arg kinectv2_enabled)">
+      <xacro:sensor_arch prefix="" parent="top_plate_link">
+        <origin xyz="-0.35 0.0 0.51" rpy="0.0 0.0 -3.14159265359"/>
+      </xacro:sensor_arch>
+      <!-- Attach the camera mount to the sensor arch -->
+      <joint name="camera_mount_joint" type="fixed">
+           <origin xyz="0.0 0.0 0.0" rpy="0.0 0.0 3.14159265359"/>
+           <parent link="sensor_arch_mount_link"/>
+           <child link="camera_mount_link"/>
+      </joint>
+      <!-- Spawn the kinectv2 mount link -->
+      <link name="camera_mount_link">
+        <visual>
+          <origin xyz="0.0 0.0 0.0" rpy="1.57079632679 0.0 1.57079632679"/>
+          <geometry>
+            <mesh filename="package://husky_description/meshes/accessories/kinectv2_mount.dae" />
+          </geometry>
+          <material name="LightGrey">
+            <color rgba="0.2 0.2 0.2 1.0"/>
+          </material>
+        </visual>
+        <collision>
+          <origin xyz="0.0 0.0 0.0" rpy="1.57079632679 0.0 1.57079632679"/>
+          <geometry>
+            <mesh filename="package://husky_description/meshes/accessories/kinectv2_mount.stl" />
+          </geometry>
+        </collision>
+      </link>
+      <joint name="camera_link_joint" type="fixed">
+        <origin xyz="0.028 -0.096 0.112" rpy="0.0 0.0 0.0" />
+        <parent link="camera_mount_link"/>
+        <child link="camera_link"/>
+      </joint>
+      <link name="kinect2_link" />
+      <joint name="kinect2_link_joint" type="fixed">
+        <origin xyz="0.0 0.0 0.0" rpy="-1.57079632679 0 -1.57079632679" />
+        <parent link="camera_link"/>
+        <child link="kinect2_link"/>
+      </joint>
+      <xacro:kinectv2_camera prefix="camera"/>
+    </xacro:if>
+    <!-- Spawn Primesense Carmine 1.09 if primesense_enabled = "true" -->
+    <xacro:if value="$(arg primesense_enabled)">
+      <xacro:sensor_arch prefix="" parent="top_plate_link">
+        <origin xyz="-0.35 0 0.51" rpy="0 0 -3.14159265359"/>
+      </xacro:sensor_arch>
+      <joint name="primesense_camera_joint" type="fixed">
+        <origin xyz="-0.020 0 0.0343994" rpy="0.0 0.0 3.14159265359" />
+        <parent link="sensor_arch_mount_link"/>
+        <child link="camera_link"/>
+      </joint>
+      <xacro:primesense_camera prefix="camera"/>
+      <link name="camera_rgb_frame" />
+      <joint name="camera_rgb_joint" type="fixed">
+        <origin rpy="0 0 0" xyz="0 0.02 0" />
+        <parent link="camera_link" />
+        <child link="camera_rgb_frame" />
+      </joint>
+      <link name="camera_rgb_optical_frame" />
+      <joint name="camera_rgb_optical_joint" type="fixed">
+        <origin rpy="-1.57079632679 0 -1.57079632679" xyz="0 0 0" />
+        <parent link="camera_rgb_frame" />
+        <child link="camera_rgb_optical_frame" />
+      </joint>
+      <link name="camera_depth_frame" />
+      <joint name="camera_depth_joint" type="fixed">
+        <origin rpy="0 0 0" xyz="0 0.045 0" />
+        <parent link="camera_link" />
+        <child link="camera_depth_frame" />
+      </joint>
+      <link name="camera_depth_optical_frame" />
+      <joint name="camera_depth_optical_joint" type="fixed">
+        <origin rpy="-1.57079632679 0 -1.57079632679" xyz="0 0 0" />
+        <parent link="camera_depth_frame" />
+        <child link="camera_depth_optical_frame" />
+      </joint>
     </xacro:if>
   </xacro:macro>

File: universal_robot/ur_description/urdf/ur5.urdf.xacro (robot description, xacro)
@@ -4,4 +4,5 @@
   <xacro:include filename="$(find ur_description)/urdf/ur.gazebo.xacro" />
   <property name="pi" value="3.14159265" />
+  <property name="stl_scale" value="0.001" />
   <!-- Inertia parameters -->
   <property name="base_mass" value="4.0" />  <!-- This mass might be incorrect -->
@@ -306,4 +307,69 @@
       <child link="${prefix}tool0"/>
     </joint>
+    <xacro:if value="$(arg ur5_camera_enabled)">
+      <joint name="${prefix}camera_mount_joint" type="fixed">
+        <origin xyz="0.0 ${wrist_3_length} 0.0" rpy="0.0 0.0 ${pi/2}" />
+        <parent link="${prefix}wrist_3_link" />
+        <child link = "${prefix}camera_mount_link" />
+      </joint>
+      <link name="${prefix}camera_mount_link">
+        <visual>
+          <origin xyz="0.0 0.0 0.0" rpy="0.0 0.0 0.0" />
+          <geometry>
+            <mesh filename="package://ur_description/meshes/ur5/visual/camera_mount.dae" scale="${stl_scale} ${stl_scale} ${stl_scale}"/>
+          </geometry>
+        </visual>
+        <collision>
+          <origin xyz="0.0 0.0 0.0" rpy="0.0 0.0 0.0" />
+          <geometry>
+            <mesh filename="package://ur_description/meshes/ur5/collision/camera_mount.stl" scale="${stl_scale} ${stl_scale} ${stl_scale}"/>
+          </geometry>
+        </collision>
+      </link>
+       <joint name="${prefix}camera_joint" type="fixed">
+         <origin xyz=".056433755002348 0.0 0.069206449979048" rpy="0.0 0.29984756549263 0.0" />
+         <parent link="${prefix}camera_mount_link" />
+         <child link = "${prefix}camera_link" />
+       </joint>
+       <link name="${prefix}camera_link">
+         <visual>
+           <origin xyz="-0.0295 0.0 0.0" rpy="0.0 0.0 0.0" />
+           <geometry>
+             <mesh filename="package://ur_description/meshes/ur5/visual/camera.dae" scale="${stl_scale} ${stl_scale} ${stl_scale}"/>
+           </geometry>
+         </visual>
+         <collision>
+           <origin xyz="-0.0295 0.0 0.0" rpy="0.0 0.0 0.0" />
+           <geometry>
+             <mesh filename="package://ur_description/meshes/ur5/collision/camera.stl" scale="${stl_scale} ${stl_scale} ${stl_scale}"/>
+           </geometry>
+         </collision>
+       </link>
+       <link name="${prefix}camera_optical_frame"/>
+       <joint name="${prefix}camera_optical_joint" type="fixed">
+          <origin xyz="0.0 0.0 0.0" rpy="-1.5708 0.0 -1.5708"/>
+          <parent link="${prefix}camera_link"/>
+          <child link="${prefix}camera_optical_frame"/>
+      </joint>
+       <joint name="${prefix}laser_pointer_joint" type="fixed">
+         <origin xyz="0.157 0.0 0.0" rpy="0.0 0.0 0.0" />
+         <parent link="${prefix}camera_mount_link" />
+         <child link = "${prefix}laser_pointer_link" />
+       </joint>
+       <link name="${prefix}laser_pointer_link">
+         <visual>
+           <origin xyz="-0.157 0.0 0.0" rpy="0.0 0.0 0.0" />
+           <geometry>
+             <mesh filename="package://ur_description/meshes/ur5/visual/laser_pointer.dae" scale="${stl_scale} ${stl_scale} ${stl_scale}"/>
+           </geometry>
+         </visual>
+         <collision>
+           <origin xyz="-0.157 0.0 0.0" rpy="0.0 0.0 0.0" />
+           <geometry>
+             <mesh filename="package://ur_description/meshes/ur5/collision/laser_pointer.stl" scale="${stl_scale} ${stl_scale} ${stl_scale}"/>
+           </geometry>
+         </collision>
+       </link>
+    </xacro:if>
   </xacro:macro>
 </robot>
