Commit message: Update packages so gripper can move.

File: husky/husky_description/urdf/husky.urdf.xacro (robot description, xacro)
@@ -29,4 +29,5 @@
   <xacro:include filename="$(find husky_description)/urdf/accessories/sensor_arch.urdf.xacro"/>
   <xacro:include filename="$(find ur_description)/urdf/ur5.urdf.xacro" />
+  <xacro:include filename="$(find mybot_description)/urdf/gripper.xacro" />
   <property name="M_PI" value="3.14159"/>
   <!-- Base Size -->
@@ -73,7 +74,7 @@
     <link name="inertial_link">
       <inertial>
-        <mass value="33.455" />
+        <mass value="330.455" />
         <origin xyz="-0.08748 -0.00085 0.09947" />
-        <inertia ixx="0.6022" ixy="-0.02364" ixz="-0.1197" iyy="1.7386" iyz="-0.001544" izz="2.0296" />
+        <inertia ixx="10.6022" ixy="-0.02364" ixz="-0.1197" iyy="10.7386" iyz="-0.001544" izz="20.0296" />
       </inertial>
     </link>
@@ -117,4 +118,12 @@
         <origin xyz="0.3058 0 0.0065" rpy="0.0 0.0 -1.57" />
       </joint>
+      <!-- Spawn gripper-->
+      <xacro:gripper />
+      <!-- Join Gripper -->
+        <joint name="base_to_arm" type="fixed">
+          <parent link="ur5_arm_wrist_3_link"/>
+          <child link="base"/>
+          <origin xyz="0 0.09 0" rpy="0 0 0"/>
+        </joint>
     </xacro:if>
     <xacro:if value="$(arg laser_enabled)">

File: universal_robot/ur_description/urdf/ur5.urdf.xacro (robot description, xacro)
@@ -306,156 +306,4 @@
       <child link="${prefix}tool0"/>
     </joint>
-    <!-- Mount for end gripper effector -->
-  <!-- xacro:if value="$(arg gripper_enabled)" -->
-    <joint name="${prefix}base_gripper_joint" type="fixed">
-      <parent link="${prefix}wrist_3_link" />
-      <child link = "${prefix}base_gripper_link" />
-      <origin xyz="0.0 ${wrist_3_length} 0.0" rpy="0.0 0.0 0.0" />
-    </joint>
-    <link name="${prefix}base_gripper_link">
-      <visual>
-        <geometry>
-          <mesh filename="package://ur_description/meshes/ur5/visual/base_grip.DAE" />
-        </geometry>
-        <material name="LightGrey">
-          <color rgba="0.7 0.7 0.7 1.0"/>
-        </material>
-      </visual>
-      <collision>
-        <geometry>
-          <mesh filename="package://ur_description/meshes/ur5/visual/base_grip.DAE" />
-        </geometry>
-      </collision>
-      <xacro:cylinder_inertial radius="0.55" length="0.02" mass="0.02">
-        <origin xyz="0.0 0.0 0.0" rpy="0 0 0" />
-      </xacro:cylinder_inertial>
-    </link>
-    <!-- Link from base gripper to gripper -->
-    <joint name="${prefix}cross_joint" type="fixed">
-      <parent link="${prefix}base_gripper_link" />
-      <child link = "${prefix}cross_link" />
-      <origin xyz="0.0 0.008 -0.07" rpy="0.0 0.0 ${pi/2}" />
-    </joint>
-    <link name="${prefix}cross_link">
-      <visual>
-        <geometry>
-          <mesh filename="package://ur_description/meshes/ur5/visual/link1.DAE" />
-        </geometry>
-        <material name="LightGrey">
-          <color rgba="0.7 0.7 0.7 1.0"/>
-        </material>
-      </visual>
-      <collision>
-        <geometry>
-          <mesh filename="package://ur_description/meshes/ur5/visual/link1.DAE" />
-        </geometry>
-      </collision>
-    </link>
-    <!-- Motor box -->
-    <joint name="${prefix}motor_joint" type="fixed">
-      <parent link="${prefix}base_gripper_link" />
-      <child link = "${prefix}motor_link" />
-      <origin xyz="0.0 0.0 -0.07" rpy="${pi/2} ${pi/2} 0.0" />
-    </joint>
-    <link name="${prefix}motor_link">
-      <visual>
-        <geometry>
-          <mesh filename="package://ur_description/meshes/ur5/visual/motor.dae" />
-        </geometry>
-        <material name="LightGrey">
-          <color rgba="0.7 0.7 0.7 1.0"/>
-        </material>
-      </visual>
-      <collision>
-        <geometry>
-          <mesh filename="package://ur_description/meshes/ur5/collision/motor.stl" />
-        </geometry>
-      </collision>
-    </link>
-   <!-- Gripper box -->
-    <joint name="${prefix}gripper_joint" type="fixed">
-      <parent link="${prefix}cross_link" />
-      <child link = "${prefix}gripper_link" />
-      <origin xyz="0.105 0.0 0.0" rpy="0.0 0.0 ${-pi/2}" />
-    </joint>
-    <link name="${prefix}gripper_link">
-      <visual>
-        <geometry>
-          <mesh filename="package://ur_description/meshes/ur5/visual/link2.DAE" />
-        </geometry>
-        <material name="LightGrey">
-          <color rgba="0.7 0.7 0.7 1.0"/>
-        </material>
-      </visual>
-      <collision>
-        <geometry>
-          <mesh filename="package://ur_description/meshes/ur5/visual/link2.DAE" />
-        </geometry>
-      </collision>
-    </link>
-    <!-- Right gripper -->
-    <joint name="${prefix}r_grip_joint" type="fixed">
-      <parent link="${prefix}gripper_link" />
-      <child link = "${prefix}r_grip_link" />
-      <origin xyz="-0.012 -0.001 0.0" rpy="0.0 0.0 ${3*pi/4}" />
-    </joint>
-    <link name="${prefix}r_grip_link">
-      <visual>
-        <geometry>
-          <mesh filename="package://ur_description/meshes/ur5/visual/tip.DAE" />
-        </geometry>
-        <material name="LightGrey">
-          <color rgba="0.7 0.7 0.7 1.0"/>
-        </material>
-      </visual>
-      <collision>
-        <geometry>
-          <mesh filename="package://ur_description/meshes/ur5/visual/tip.DAE" />
-        </geometry>
-      </collision>
-    </link>
-    <!-- Left gripper -->
-    <joint name="${prefix}l_grip_joint" type="fixed">
-      <parent link="${prefix}gripper_link" />
-      <child link = "${prefix}l_grip_link" />
-      <origin xyz="0.012 0.00 0.0" rpy="${pi} 0.0 ${9*pi/4}" />
-    </joint>
-    <link name="${prefix}l_grip_link">
-      <visual>
-        <geometry>
-          <mesh filename="package://ur_description/meshes/ur5/visual/tip.DAE" />
-        </geometry>
-        <material name="LightGrey">
-          <color rgba="0.7 0.7 0.7 1.0"/>
-        </material>
-      </visual>
-      <collision>
-        <geometry>
-          <mesh filename="package://ur_description/meshes/ur5/visual/tip.DAE" />
-        </geometry>
-      </collision>
-    </link>
-    <!-- On arm camera -->
-    <joint name="${prefix}depthsense_joint" type="fixed">
-      <parent link="${prefix}base_gripper_link" />
-      <child link = "${prefix}depthsense_link" />
-      <origin xyz="0.0 0.005 0.0" rpy="${pi/2} 0.0 ${pi}" />
-    </joint>
-    <link name="${prefix}depthsense_link">
-      <visual>
-        <geometry>
-          <mesh filename="package://ur_description/meshes/ur5/visual/depthsense.dae" />
-        </geometry>
-        <material name="LightGrey">
-          <color rgba="0.7 0.7 0.7 1.0"/>
-        </material>
-      </visual>
-      <collision>
-        <geometry>
-          <mesh filename="package://ur_description/meshes/ur5/collision/depthsense.stl" />
-        </geometry>
-      </collision>
-    </link>
-    <!-- /xacro:if -->
   </xacro:macro>
 </robot>

Commit message: Updated orient package to work with updated Husky.

File: husky/husky_description/urdf/husky.urdf.xacro (robot description, xacro)
@@ -76,5 +76,5 @@
     <link name="inertial_link">
       <inertial>
-        <mass value="80" />
+        <mass value="60" />
         <origin xyz="-0.08748 -0.00085 0.09947" />
         <inertia ixx="1.08995475113" ixy="-0.0427873303" ixz="-0.2166515837" iyy="3.14678733031" iyz="-0.00279457012" izz="3.67348416289" />

Commit message: Partial fix for new husky model.

File: husky/husky_description/urdf/husky.urdf.xacro (robot description, xacro)
@@ -80,5 +80,5 @@
         <inertia ixx="1.08995475113" ixy="-0.0427873303" ixz="-0.2166515837" iyy="3.14678733031" iyz="-0.00279457012" izz="3.67348416289" />
       </inertial>
-    </link>
+</link>
     <joint name="inertial_joint" type="fixed">
       <origin xyz="0 0 0" rpy="0 0 0" />

Commit message: Updated to current, added param manipulation

File: husky/husky_description/urdf/husky.urdf.xacro (robot description, xacro)
@@ -76,6 +76,9 @@
     <link name="inertial_link">
       <inertial>
+        <!-- <mass value="33.455" /> -->
         <mass value="60" />
+        <!-- <origin xyz="-0.08748 -0.00085 -0.2" /> -->
         <origin xyz="-0.08748 -0.00085 0.09947" />
+        <!-- <inertia ixx="1.0" ixy="0.0" ixz="0.0" iyy="1.0" iyz="0.0" izz="1.0" /> -->
         <inertia ixx="1.08995475113" ixy="-0.0427873303" ixz="-0.2166515837" iyy="3.14678733031" iyz="-0.00279457012" izz="3.67348416289" />
       </inertial>

File: universal_robot/ur_description/urdf/ur5.urdf.xacro (robot description, xacro)
@@ -91,5 +91,6 @@
       <parent link="${prefix}base_link" />
       <child link = "${prefix}shoulder_link" />
-      <origin xyz="0.0 0.0 ${shoulder_height}" rpy="0.0 0.0 0.0" />
+      <origin xyz="0.0 0.0 ${shoulder_height}" rpy="0.0 0.0 1.5707" />
+      <!-- <origin xyz="0.0 0.0 ${shoulder_height}" rpy="0.0 0.0 0.0" /> -->
       <axis xyz="0 0 1" />
       <xacro:unless value="${joint_limited}">
@@ -122,5 +123,10 @@
       <parent link="${prefix}shoulder_link" />
       <child link = "${prefix}upper_arm_link" />
-      <origin xyz="0.0 ${shoulder_offset} 0.0" rpy="0.0 ${pi / 2.0} 0.0" />
+      <!-- Test arm forward -->
+      <!-- <origin xyz="0.0 ${shoulder_offset} 0.0" rpy="0.0 ${pi / 4} 0.0" /> -->
+      <!-- Stow position flat -->
+      <!-- <origin xyz="0.0 ${shoulder_offset} 0.0" rpy="0.0 -1.5707 0.0" /> -->
+      <!-- Stow position up -->
+      <origin xyz="0.0 ${shoulder_offset} 0.0" rpy="0.0 -1.122 0.0" />
       <axis xyz="0 1 0" />
       <xacro:unless value="${joint_limited}">
@@ -153,5 +159,8 @@
       <parent link="${prefix}upper_arm_link" />
       <child link = "${prefix}forearm_link" />
-      <origin xyz="0.0 ${elbow_offset} ${upper_arm_length}" rpy="0.0 0.0 0.0" />
+      <!-- Test arm forward -->
+      <!-- <origin xyz="0.0 ${elbow_offset} ${upper_arm_length}" rpy="0.0 ${pi / 4} 0.0" /> -->
+      <!-- Stow position -->
+      <origin xyz="0.0 ${elbow_offset} ${upper_arm_length}" rpy="0.0 2.6927 0.0" />
       <axis xyz="0 1 0" />
       <xacro:unless value="${joint_limited}">
@@ -184,5 +193,10 @@
       <parent link="${prefix}forearm_link" />
       <child link = "${prefix}wrist_1_link" />
-      <origin xyz="0.0 0.0 ${forearm_length}" rpy="0.0 ${pi / 2.0} 0.0" />
+      <!-- Test arm forward -->
+      <!-- <origin xyz="0.0 0.0 ${forearm_length}" rpy="0.0 -1.5707 0.0" /> -->
+      <!-- Stow position flat -->
+      <!-- <origin xyz="0.0 0.0 ${forearm_length}" rpy="0.0 -1.122 0.0" /> -->
+      <!-- Stow position up -->
+      <origin xyz="0.0 0.0 ${forearm_length}" rpy="0.0 -1.5707 0.0" />
       <axis xyz="0 1 0" />
       <xacro:unless value="${joint_limited}">
@@ -215,5 +229,6 @@
       <parent link="${prefix}wrist_1_link" />
       <child link = "${prefix}wrist_2_link" />
-      <origin xyz="0.0 ${wrist_1_length} 0.0" rpy="0.0 0.0 0.0" />
+      <origin xyz="0.0 ${wrist_1_length} 0.0" rpy="0.0 0.0 -1.5707" />
+      <!-- <origin xyz="0.0 ${wrist_1_length} 0.0" rpy="0.0 0.0 0.0" /> -->
       <axis xyz="0 0 1" />
       <xacro:unless value="${joint_limited}">
@@ -247,4 +262,5 @@
       <child link = "${prefix}wrist_3_link" />
       <origin xyz="0.0 0.0 ${wrist_2_length}" rpy="0.0 0.0 0.0" />
+      <!-- <origin xyz="0.0 0.0 ${wrist_2_length}" rpy="0.0 0.0 0.0" /> -->
       <axis xyz="0 1 0" />
       <xacro:unless value="${joint_limited}">
