Commit message: Updated husky_description urdfs to include gripper, need to incorp Tom c

File: husky/husky_description/urdf/description.xacro (robot description, xacro)
@@ -22,9 +22,10 @@
 -->
 <robot name="husky" xmlns:xacro="http://ros.org/wiki/xacro">
-  <xacro:arg name="laser_enabled" default="false" />
+  <xacro:arg name="laser_enabled" default="true" />
   <xacro:arg name="ur5_enabled" default="false" />
   <xacro:arg name="ur5_camera_enabled" default="false" />
+  <xacro:arg name="ur5_mbzirc_gripper_enabled" default="true" />
   <xacro:arg name="kinect_enabled" default="false" />
-  <xacro:arg name="kinectv2_enabled" default="false" />
+  <xacro:arg name="kinectv2_enabled" default="true" />
   <xacro:arg name="primesense_enabled" default="false"/>
   <xacro:include filename="$(find husky_description)/urdf/husky.urdf.xacro" />

File: husky/husky_description/urdf/husky.urdf.xacro (robot description, xacro)
@@ -31,5 +31,4 @@
   <xacro:include filename="$(find husky_description)/urdf/accessories/sensor_arch.urdf.xacro"/>
   <xacro:include filename="$(find ur_description)/urdf/ur5.urdf.xacro" />
-  <xacro:include filename="$(find mybot_description)/urdf/gripper.xacro" />
   <property name="M_PI" value="3.14159"/>
   <!-- Base Size -->
@@ -76,12 +75,9 @@
     <link name="inertial_link">
       <inertial>
-        <!-- <mass value="33.455" /> -->
         <mass value="60" />
-        <!-- <origin xyz="-0.08748 -0.00085 -0.2" /> -->
         <origin xyz="-0.08748 -0.00085 0.09947" />
-        <!-- <inertia ixx="1.0" ixy="0.0" ixz="0.0" iyy="1.0" iyz="0.0" izz="1.0" /> -->
         <inertia ixx="1.08995475113" ixy="-0.0427873303" ixz="-0.2166515837" iyy="3.14678733031" iyz="-0.00279457012" izz="3.67348416289" />
       </inertial>
-</link>
+    </link>
     <joint name="inertial_joint" type="fixed">
       <origin xyz="0 0 0" rpy="0 0 0" />
@@ -123,14 +119,17 @@
         <origin xyz="0.3058 0 0.0065" rpy="0.0 0.0 -1.57079632679" />
       </joint>
-      <!-- Spawn gripper-->
-      <xacro:gripper />
-      <!-- Join Gripper -->
-        <joint name="base_to_arm" type="fixed">
-          <parent link="ur5_arm_wrist_3_link"/>
-          <child link="base"/>
-          <origin xyz="0 0.09 0" rpy="0 0 0"/>
-        </joint>
     </xacro:if>
     <xacro:if value="$(arg ur5_camera_enabled)">
+      <xacro:property name="reflect" value="-1" />
+      <!-- Spawn arm -->
+      <xacro:ur5_robot prefix="ur5_arm_" joint_limited="true"/>
+      <!-- Join arm -->
+      <joint name="ur5_arm_base" type="fixed">
+        <parent link="top_plate_link" />
+        <child link="ur5_arm_base_link" />
+        <origin xyz="0.3058 0 0.0065" rpy="0.0 0.0 -1.57079632679" />
+      </joint>
+    </xacro:if>
+    <xacro:if value="$(arg ur5_mbzirc_gripper_enabled)">
       <xacro:property name="reflect" value="-1" />
       <!-- Spawn arm -->

File: husky/husky_description/urdf/husky_ur5.urdf (robot description, URDF)
Before this commit: robot husky, 32 links, 31 joints
Links:
- removed link camera_optical_frame
- removed link ur5_arm_camera_link
- removed link ur5_arm_camera_mount_link
- removed link ur5_arm_camera_optical_frame
- removed link ur5_arm_laser_pointer_link
- added link kinect2_link
- added link ur5_arm_gripper_base_link, mass 2.7; collision mesh filename=package://gripper_description/meshes/base_link.stl scale=0.001 0.001 0.001; visual mesh filename=package://gripper_description/meshes/base_link.dae scale=0.001 0.001 0.001
- added link ur5_arm_gripper_camera_link, mass 0.05; collision box size=0.05 0.0125 0.0125; visual box size=0.05 0.025 0.0125
- added link ur5_arm_gripper_camera_optical_frame
- added link ur5_arm_gripper_left_tip, mass 2.07; collision mesh filename=package://gripper_description/meshes/tip.stl scale=0.001 0.001 0.001; visual mesh filename=package://gripper_description/meshes/tip.dae scale=0.001 0.001 0.001
- added link ur5_arm_gripper_link_1, mass 2.9; collision mesh filename=package://gripper_description/meshes/link_1.stl scale=0.001 0.001 0.001; visual mesh filename=package://gripper_description/meshes/link_1.dae scale=0.001 0.001 0.001
- added link ur5_arm_gripper_link_2, mass 2.2; collision mesh filename=package://gripper_description/meshes/link_2.stl scale=0.001 0.001 0.001; visual mesh filename=package://gripper_description/meshes/link_2.dae scale=0.001 0.001 0.001
- added link ur5_arm_gripper_right_tip, mass 2.07; collision mesh filename=package://gripper_description/meshes/tip.stl scale=0.001 0.001 0.001; visual mesh filename=package://gripper_description/meshes/tip.dae scale=0.001 0.001 0.001
- link inertial_link: mass 33.455 -> 60
Joints:
- removed joint camera_optical_joint
- removed joint kinectv2_frame_joint
- removed joint ur5_arm_camera_joint
- removed joint ur5_arm_camera_mount_joint
- removed joint ur5_arm_camera_optical_joint
- removed joint ur5_arm_laser_pointer_joint
- added joint camera_link_joint: type fixed, parent camera_mount_link, child camera_link, origin xyz=0.028 -0.096 0.112 rpy=0.0 0.0 0.0
- added joint kinect2_link_joint: type fixed, parent camera_link, child kinect2_link, origin xyz=0.0 0.0 0.0 rpy=-1.57079632679 0 -1.57079632679
- added joint ur5_arm_gripper_base_link_camera_joint: type fixed, parent ur5_arm_gripper_base_link, child ur5_arm_gripper_camera_link, origin xyz=0 0 0 rpy=0 0 0
- added joint ur5_arm_gripper_base_link_link_1_joint: type fixed, parent ur5_arm_gripper_base_link, child ur5_arm_gripper_link_1, origin xyz=0 0.005 -0.07 rpy=0 0 1.57079632679
- added joint ur5_arm_gripper_camera_optical_joint: type fixed, parent ur5_arm_gripper_camera_link, child ur5_arm_gripper_camera_optical_frame, origin xyz=0 0 0 rpy=-1.57079632679 0 -1.57079632679
- added joint ur5_arm_gripper_link_1_link_2_joint: type fixed, parent ur5_arm_gripper_link_1, child ur5_arm_gripper_link_2, origin xyz=0.104 0 0 rpy=0 0 1.57079632679
- added joint ur5_arm_gripper_link_2_left_tip_joint: type revolute, parent ur5_arm_gripper_link_2, child ur5_arm_gripper_left_tip, origin xyz=0.0125 0 0.00025 rpy=0 0 -1.57079632679, axis 0 0 1, limit lower=-0.037 upper=0.6 effort=100 velocity=5
- added joint ur5_arm_gripper_link_2_right_tip_joint: type revolute, parent ur5_arm_gripper_link_2, child ur5_arm_gripper_right_tip, origin xyz=-0.0125 0 0.00025 rpy=0 0 1.57079632679, axis 0 0 1, limit lower=-0.6 upper=0.037 effort=100 velocity=5
- added joint ur5_arm_gripper_wrist_3_link_gripper_base_link_joint: type fixed, parent ur5_arm_wrist_3_link, child ur5_arm_gripper_base_link, origin xyz=0.0 0.0823 0.0 rpy=0.0 0.0 0.0
- joint base_laser_joint: origin xyz=-0.0352 0 -0.0566 rpy=3.14159 0 0 -> xyz=-0.0352 0 -0.0566 rpy=0 0 0
- joint camera_mount_joint: origin xyz=0.0 0.0 0.0 rpy=0.0 0.0 0.0 -> xyz=0.0 0.0 0.0 rpy=0.0 0.0 3.14159265359
- joint imu_joint: origin xyz=0.19 0 0.149 rpy=0 -1.5708 3.14159265359 -> xyz=0.19 0 0.149 rpy=0 -1.57079632679 3.14159265359
- joint ur5_arm_base: origin xyz=0.3058 0 0.0065 rpy=0.0 0.0 -1.57 -> xyz=0.3058 0 0.0065 rpy=0.0 0.0 -1.57079632679
- joint ur5_arm_elbow_joint: origin xyz=0.0 -0.1197 0.425 rpy=0.0 0.0 0.0 -> xyz=0.0 -0.1197 0.425 rpy=0.0 2.6927 0.0
- joint ur5_arm_shoulder_lift_joint: origin xyz=0.0 0.13585 0.0 rpy=0.0 1.570796325 0.0 -> xyz=0.0 0.13585 0.0 rpy=0.0 -1.122 0.0
- joint ur5_arm_shoulder_pan_joint: origin xyz=0.0 0.0 0.089159 rpy=0.0 0.0 0.0 -> xyz=0.0 0.0 0.089159 rpy=0.0 0.0 1.5707
- joint ur5_arm_wrist_1_joint: origin xyz=0.0 0.0 0.39225 rpy=0.0 1.570796325 0.0 -> xyz=0.0 0.0 0.39225 rpy=0.0 -1.5707 0.0
- joint ur5_arm_wrist_2_joint: origin xyz=0.0 0.093 0.0 rpy=0.0 0.0 0.0 -> xyz=0.0 0.093 0.0 rpy=0.0 0.0 -1.5707

Commit message: Revert "URDF fix and added submodule"

File: husky/husky_description/urdf/description.xacro (robot description, xacro)
@@ -22,10 +22,9 @@
 -->
 <robot name="husky" xmlns:xacro="http://ros.org/wiki/xacro">
-  <xacro:arg name="laser_enabled" default="true" />
+  <xacro:arg name="laser_enabled" default="false" />
   <xacro:arg name="ur5_enabled" default="false" />
   <xacro:arg name="ur5_camera_enabled" default="false" />
-  <xacro:arg name="ur5_mbzirc_gripper_enabled" default="true" />
   <xacro:arg name="kinect_enabled" default="false" />
-  <xacro:arg name="kinectv2_enabled" default="true" />
+  <xacro:arg name="kinectv2_enabled" default="false" />
   <xacro:arg name="primesense_enabled" default="false"/>
   <xacro:include filename="$(find husky_description)/urdf/husky.urdf.xacro" />

File: husky/husky_description/urdf/husky.urdf.xacro (robot description, xacro)
@@ -31,4 +31,5 @@
   <xacro:include filename="$(find husky_description)/urdf/accessories/sensor_arch.urdf.xacro"/>
   <xacro:include filename="$(find ur_description)/urdf/ur5.urdf.xacro" />
+  <xacro:include filename="$(find mybot_description)/urdf/gripper.xacro" />
   <property name="M_PI" value="3.14159"/>
   <!-- Base Size -->
@@ -75,9 +76,12 @@
     <link name="inertial_link">
       <inertial>
+        <!-- <mass value="33.455" /> -->
         <mass value="60" />
+        <!-- <origin xyz="-0.08748 -0.00085 -0.2" /> -->
         <origin xyz="-0.08748 -0.00085 0.09947" />
+        <!-- <inertia ixx="1.0" ixy="0.0" ixz="0.0" iyy="1.0" iyz="0.0" izz="1.0" /> -->
         <inertia ixx="1.08995475113" ixy="-0.0427873303" ixz="-0.2166515837" iyy="3.14678733031" iyz="-0.00279457012" izz="3.67348416289" />
       </inertial>
-    </link>
+</link>
     <joint name="inertial_joint" type="fixed">
       <origin xyz="0 0 0" rpy="0 0 0" />
@@ -119,17 +123,14 @@
         <origin xyz="0.3058 0 0.0065" rpy="0.0 0.0 -1.57079632679" />
       </joint>
+      <!-- Spawn gripper-->
+      <xacro:gripper />
+      <!-- Join Gripper -->
+        <joint name="base_to_arm" type="fixed">
+          <parent link="ur5_arm_wrist_3_link"/>
+          <child link="base"/>
+          <origin xyz="0 0.09 0" rpy="0 0 0"/>
+        </joint>
     </xacro:if>
     <xacro:if value="$(arg ur5_camera_enabled)">
-      <xacro:property name="reflect" value="-1" />
-      <!-- Spawn arm -->
-      <xacro:ur5_robot prefix="ur5_arm_" joint_limited="true"/>
-      <!-- Join arm -->
-      <joint name="ur5_arm_base" type="fixed">
-        <parent link="top_plate_link" />
-        <child link="ur5_arm_base_link" />
-        <origin xyz="0.3058 0 0.0065" rpy="0.0 0.0 -1.57079632679" />
-      </joint>
-    </xacro:if>
-    <xacro:if value="$(arg ur5_mbzirc_gripper_enabled)">
       <xacro:property name="reflect" value="-1" />
       <!-- Spawn arm -->

File: husky/husky_description/urdf/husky_ur5.urdf (robot description, URDF)
Before this commit: robot husky, 35 links, 34 joints
Links:
- removed link kinect2_link
- removed link ur5_arm_gripper_base_link
- removed link ur5_arm_gripper_camera_link
- removed link ur5_arm_gripper_camera_optical_frame
- removed link ur5_arm_gripper_left_tip
- removed link ur5_arm_gripper_link_1
- removed link ur5_arm_gripper_link_2
- removed link ur5_arm_gripper_right_tip
- added link camera_optical_frame
- added link ur5_arm_camera_link; collision mesh filename=package://ur_description/meshes/ur5/collision/camera.stl scale=0.001 0.001 0.001; visual mesh filename=package://ur_description/meshes/ur5/visual/camera.dae scale=0.001 0.001 0.001
- added link ur5_arm_camera_mount_link; collision mesh filename=package://ur_description/meshes/ur5/collision/camera_mount.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 scale=0.001 0.001 0.001; visual mesh filename=package://ur_description/meshes/ur5/visual/camera_mount.dae scale=0.001 0.001 0.001
- added link ur5_arm_camera_optical_frame
- added link ur5_arm_laser_pointer_link; collision mesh filename=package://ur_description/meshes/ur5/collision/laser_pointer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 scale=0.001 0.001 0.001; visual mesh filename=package://ur_description/meshes/ur5/visual/laser_pointer.dae scale=0.001 0.001 0.001
- link inertial_link: mass 60 -> 33.455
Joints:
- removed joint camera_link_joint
- removed joint kinect2_link_joint
- removed joint ur5_arm_gripper_base_link_camera_joint
- removed joint ur5_arm_gripper_base_link_link_1_joint
- removed joint ur5_arm_gripper_camera_optical_joint
- removed joint ur5_arm_gripper_link_1_link_2_joint
- removed joint ur5_arm_gripper_link_2_left_tip_joint
- removed joint ur5_arm_gripper_link_2_right_tip_joint
- removed joint ur5_arm_gripper_wrist_3_link_gripper_base_link_joint
- added joint camera_optical_joint: type fixed, parent camera_link, child camera_optical_frame, origin xyz=0 0 0 rpy=-1.57079632679 0 -1.57079632679
- added joint kinectv2_frame_joint: type fixed, parent camera_mount_link, child camera_link, origin xyz=0.0 0.095 0.11 rpy=0.0 0.0 3.14159265359
- added joint ur5_arm_camera_joint: type fixed, parent ur5_arm_camera_mount_link, child ur5_arm_camera_link, origin xyz=.056433755002348 0.0 0.069206449979048 rpy=0.0 0.29984756549263 0.0
- added joint ur5_arm_camera_mount_joint: type fixed, parent ur5_arm_wrist_3_link, child ur5_arm_camera_mount_link, origin xyz=0.0 0.0823 0.0 rpy=0.0 0.0 1.570796325
- added joint ur5_arm_camera_optical_joint: type fixed, parent ur5_arm_camera_link, child ur5_arm_camera_optical_frame, origin xyz=0.0 0.0 0.0 rpy=-1.5708 0.0 -1.5708
- added joint ur5_arm_laser_pointer_joint: type fixed, parent ur5_arm_camera_mount_link, child ur5_arm_laser_pointer_link, origin xyz=0.157 0.0 0.0 rpy=0.0 0.0 0.0
- joint base_laser_joint: origin xyz=-0.0352 0 -0.0566 rpy=0 0 0 -> xyz=-0.0352 0 -0.0566 rpy=3.14159 0 0
- joint camera_mount_joint: origin xyz=0.0 0.0 0.0 rpy=0.0 0.0 3.14159265359 -> xyz=0.0 0.0 0.0 rpy=0.0 0.0 0.0
- joint imu_joint: origin xyz=0.19 0 0.149 rpy=0 -1.57079632679 3.14159265359 -> xyz=0.19 0 0.149 rpy=0 -1.5708 3.14159265359
- joint ur5_arm_base: origin xyz=0.3058 0 0.0065 rpy=0.0 0.0 -1.57079632679 -> xyz=0.3058 0 0.0065 rpy=0.0 0.0 -1.57
- joint ur5_arm_elbow_joint: origin xyz=0.0 -0.1197 0.425 rpy=0.0 2.6927 0.0 -> xyz=0.0 -0.1197 0.425 rpy=0.0 0.0 0.0
- joint ur5_arm_shoulder_lift_joint: origin xyz=0.0 0.13585 0.0 rpy=0.0 -1.122 0.0 -> xyz=0.0 0.13585 0.0 rpy=0.0 1.570796325 0.0
- joint ur5_arm_shoulder_pan_joint: origin xyz=0.0 0.0 0.089159 rpy=0.0 0.0 1.5707 -> xyz=0.0 0.0 0.089159 rpy=0.0 0.0 0.0
- joint ur5_arm_wrist_1_joint: origin xyz=0.0 0.0 0.39225 rpy=0.0 -1.5707 0.0 -> xyz=0.0 0.0 0.39225 rpy=0.0 1.570796325 0.0
- joint ur5_arm_wrist_2_joint: origin xyz=0.0 0.093 0.0 rpy=0.0 0.0 -1.5707 -> xyz=0.0 0.093 0.0 rpy=0.0 0.0 0.0

File: husky/husky_simulator/husky_gazebo/urdf/description.gazebo.xacro (robot description, xacro)
@@ -23,8 +23,7 @@
 <robot name="husky" xmlns:xacro="http://ros.org/wiki/xacro">
 <!-- <robot name="husky_robot_gazebo" xmlns:xacro="http://ros.org/wiki/xacro"> -->
-  <xacro:arg name="laser_enabled" default="false" />
+  <xacro:arg name="laser_enabled" default="true" />
   <xacro:arg name="ur5_enabled" default="false" />
   <xacro:arg name="ur5_camera_enabled" default="false" />
-  <xacro:arg name="ur5_mbzirc_gripper_enabled" default="false" />
   <xacro:arg name="kinect_enabled" default="false" />
   <xacro:arg name="kinectv2_enabled" default="false" />

File: husky/husky_simulator/husky_gazebo/urdf/husky.gazebo.xacro (robot description, xacro)
@@ -118,49 +118,4 @@
       </gazebo>
     </xacro:if>
-    <xacro:if value="$(arg ur5_mbzirc_gripper_enabled)">
-      <!--Remove when https://github.com/ros-industrial/universal_robot/pull/168 is resolved -->
-      <gazebo reference="ur5_arm_shoulder_link">
-        <selfCollide>true</selfCollide>
-      </gazebo>
-      <gazebo reference="ur5_arm_upper_arm_link">
-        <selfCollide>true</selfCollide>
-      </gazebo>
-      <gazebo reference="ur5_arm_forearm_link">
-        <selfCollide>true</selfCollide>
-      </gazebo>
-      <gazebo reference="ur5_arm_wrist_1_link">
-        <selfCollide>true</selfCollide>
-      </gazebo>
-      <gazebo reference="ur5_arm_wrist_3_link">
-       <selfCollide>true</selfCollide>
-      </gazebo>
-      <gazebo reference="ur5_arm_wrist_2_link">
-        <selfCollide>true</selfCollide>
-      </gazebo>
-      <gazebo reference="ur5_arm_ee_link">
-        <selfCollide>true</selfCollide>
-      </gazebo>
-      <gazebo reference="ur5_arm_gripper_base_link">
-        <selfCollide>true</selfCollide>
-      </gazebo>
-      <gazebo reference="ur5_arm_gripper_link_1">
-        <selfCollide>true</selfCollide>
-      </gazebo>
-      <gazebo reference="ur5_arm_gripper_link_2">
-        <selfCollide>true</selfCollide>
-      </gazebo>
-      <gazebo reference="ur5_arm_gripper_left_tip">
-        <selfCollide>true</selfCollide>
-      </gazebo>
-      <gazebo reference="ur5_arm_gripper_right_tip">
-        <selfCollide>true</selfCollide>
-      </gazebo>
-      <gazebo reference="ur5_arm_gripper_camera_link">
-        <selfCollide>true</selfCollide>
-      </gazebo>
-      <gazebo reference="ur5_arm_gripper_camera_optical_frame">
-        <selfCollide>true</selfCollide>
-      </gazebo>
-    </xacro:if>
     <xacro:if value="$(arg kinect_enabled)">
       <xacro:kinect_camera_gazebo prefix="camera"/>

File: universal_robot/ur_description/urdf/ur5.urdf.xacro (robot description, xacro)
@@ -3,5 +3,4 @@
   <xacro:include filename="$(find ur_description)/urdf/ur.transmission.xacro" />
   <xacro:include filename="$(find ur_description)/urdf/ur.gazebo.xacro" />
-  <xacro:include filename="$(find gripper_description)/urdf/gripper.urdf.xacro" />
   <property name="pi" value="3.14159265" />
   <property name="stl_scale" value="0.001" />
@@ -92,5 +91,6 @@
       <parent link="${prefix}base_link" />
       <child link = "${prefix}shoulder_link" />
-      <origin xyz="0.0 0.0 ${shoulder_height}" rpy="0.0 0.0 0.0" />
+      <origin xyz="0.0 0.0 ${shoulder_height}" rpy="0.0 0.0 1.5707" />
+      <!-- <origin xyz="0.0 0.0 ${shoulder_height}" rpy="0.0 0.0 0.0" /> -->
       <axis xyz="0 0 1" />
       <xacro:unless value="${joint_limited}">
@@ -123,5 +123,10 @@
       <parent link="${prefix}shoulder_link" />
       <child link = "${prefix}upper_arm_link" />
-      <origin xyz="0.0 ${shoulder_offset} 0.0" rpy="0.0 ${pi / 2.0} 0.0" />
+      <!-- Test arm forward -->
+      <!-- <origin xyz="0.0 ${shoulder_offset} 0.0" rpy="0.0 ${pi / 4} 0.0" /> -->
+      <!-- Stow position flat -->
+      <!-- <origin xyz="0.0 ${shoulder_offset} 0.0" rpy="0.0 -1.5707 0.0" /> -->
+      <!-- Stow position up -->
+      <origin xyz="0.0 ${shoulder_offset} 0.0" rpy="0.0 -1.122 0.0" />
       <axis xyz="0 1 0" />
       <xacro:unless value="${joint_limited}">
@@ -154,5 +159,8 @@
       <parent link="${prefix}upper_arm_link" />
       <child link = "${prefix}forearm_link" />
-      <origin xyz="0.0 ${elbow_offset} ${upper_arm_length}" rpy="0.0 0.0 0.0" />
+      <!-- Test arm forward -->
+      <!-- <origin xyz="0.0 ${elbow_offset} ${upper_arm_length}" rpy="0.0 ${pi / 4} 0.0" /> -->
+      <!-- Stow position -->
+      <origin xyz="0.0 ${elbow_offset} ${upper_arm_length}" rpy="0.0 2.6927 0.0" />
       <axis xyz="0 1 0" />
       <xacro:unless value="${joint_limited}">
@@ -185,5 +193,10 @@
       <parent link="${prefix}forearm_link" />
       <child link = "${prefix}wrist_1_link" />
-      <origin xyz="0.0 0.0 ${forearm_length}" rpy="0.0 ${pi / 2.0} 0.0" />
+      <!-- Test arm forward -->
+      <!-- <origin xyz="0.0 0.0 ${forearm_length}" rpy="0.0 -1.5707 0.0" /> -->
+      <!-- Stow position flat -->
+      <!-- <origin xyz="0.0 0.0 ${forearm_length}" rpy="0.0 -1.122 0.0" /> -->
+      <!-- Stow position up -->
+      <origin xyz="0.0 0.0 ${forearm_length}" rpy="0.0 -1.5707 0.0" />
       <axis xyz="0 1 0" />
       <xacro:unless value="${joint_limited}">
@@ -216,5 +229,6 @@
       <parent link="${prefix}wrist_1_link" />
       <child link = "${prefix}wrist_2_link" />
-      <origin xyz="0.0 ${wrist_1_length} 0.0" rpy="0.0 0.0 0.0" />
+      <origin xyz="0.0 ${wrist_1_length} 0.0" rpy="0.0 0.0 -1.5707" />
+      <!-- <origin xyz="0.0 ${wrist_1_length} 0.0" rpy="0.0 0.0 0.0" /> -->
       <axis xyz="0 0 1" />
       <xacro:unless value="${joint_limited}">
@@ -248,4 +262,5 @@
       <child link = "${prefix}wrist_3_link" />
       <origin xyz="0.0 0.0 ${wrist_2_length}" rpy="0.0 0.0 0.0" />
+      <!-- <origin xyz="0.0 0.0 ${wrist_2_length}" rpy="0.0 0.0 0.0" /> -->
       <axis xyz="0 1 0" />
       <xacro:unless value="${joint_limited}">
@@ -373,11 +388,4 @@
        </link>
     </xacro:if>
-    <xacro:if value="$(arg ur5_mbzirc_gripper_enabled)">
-      <joint name="${prefix}gripper_wrist_3_link_gripper_base_link_joint" type="fixed">
-        <origin xyz="0.0 ${wrist_3_length} 0.0" rpy="0.0 0.0 0.0" />
-        <parent link="${prefix}wrist_3_link" />
-        <child link="${prefix}gripper_base_link" />
-      </joint>
-    </xacro:if>
   </xacro:macro>
 </robot>
