Commit message: Balanced robot, corrected rotate command

File: husky/husky_description/urdf/husky_ur5.urdf (robot description, URDF)
Before this commit: robot husky, 32 links, 31 joints
Links:
- link sensor_arch_mount_link: mass None -> 20.0

Commit message: Adjusted urdfs and rotate command for better rotation

File: husky/husky_description/urdf/husky_ur5.urdf (robot description, URDF)
Before this commit: robot husky, 32 links, 31 joints
Joints:
- joint ur5_arm_wrist_3_joint: limit lower=-3.14159265 upper=3.14159265 effort=28.0 velocity=3.2 -> lower=-6.28318530 upper=6.28318530 effort=28.0 velocity=3.2

File: universal_robot/ur_description/urdf/ur5.urdf.xacro (robot description, xacro)
@@ -268,5 +268,5 @@
       </xacro:unless>
       <xacro:if value="${joint_limited}">
-        <limit lower="${-pi}" upper="${pi}" effort="28.0" velocity="3.2"/>
+        <limit lower="${-2.0 * pi}" upper="${2.0 * pi}" effort="28.0" velocity="3.2"/>
       </xacro:if>
       <dynamics damping="0.0" friction="0.0"/>
