Commit message: Fixed initial position of the robot

File: universal_robot/ur_description/urdf/ur5.urdf.xacro (robot description, xacro)
@@ -91,5 +91,6 @@
       <parent link="${prefix}base_link" />
       <child link = "${prefix}shoulder_link" />
-      <origin xyz="0.0 0.0 ${shoulder_height}" rpy="0.0 0.0 0.0" />
+      <origin xyz="0.0 0.0 ${shoulder_height}" rpy="0.0 0.0 1.5707" />
+      <!-- <origin xyz="0.0 0.0 ${shoulder_height}" rpy="0.0 0.0 0.0" /> -->
       <axis xyz="0 0 1" />
       <xacro:unless value="${joint_limited}">
@@ -122,5 +123,6 @@
       <parent link="${prefix}shoulder_link" />
       <child link = "${prefix}upper_arm_link" />
-      <origin xyz="0.0 ${shoulder_offset} 0.0" rpy="0.0 ${pi / 2.0} 0.0" />
+      <origin xyz="0.0 ${shoulder_offset} 0.0" rpy="0.0 -1.122 0.0" />
+      <!-- <origin xyz="0.0 ${shoulder_offset} 0.0" rpy="0.0 ${pi / 2.0} 0.0" /> -->
       <axis xyz="0 1 0" />
       <xacro:unless value="${joint_limited}">
@@ -153,5 +155,6 @@
       <parent link="${prefix}upper_arm_link" />
       <child link = "${prefix}forearm_link" />
-      <origin xyz="0.0 ${elbow_offset} ${upper_arm_length}" rpy="0.0 0.0 0.0" />
+      <origin xyz="0.0 ${elbow_offset} ${upper_arm_length}" rpy="0.0 2.6927 0.0" />
+      <!-- <origin xyz="0.0 ${elbow_offset} ${upper_arm_length}" rpy="0.0 0.0 0.0" /> -->
       <axis xyz="0 1 0" />
       <xacro:unless value="${joint_limited}">
@@ -184,5 +187,6 @@
       <parent link="${prefix}forearm_link" />
       <child link = "${prefix}wrist_1_link" />
-      <origin xyz="0.0 0.0 ${forearm_length}" rpy="0.0 ${pi / 2.0} 0.0" />
+      <origin xyz="0.0 0.0 ${forearm_length}" rpy="0.0 -1.5707 0.0" />
+      <!-- <origin xyz="0.0 0.0 ${forearm_length}" rpy="0.0 ${pi / 2.0} 0.0" /> -->
       <axis xyz="0 1 0" />
       <xacro:unless value="${joint_limited}">
@@ -215,5 +219,6 @@
       <parent link="${prefix}wrist_1_link" />
       <child link = "${prefix}wrist_2_link" />
-      <origin xyz="0.0 ${wrist_1_length} 0.0" rpy="0.0 0.0 0.0" />
+      <origin xyz="0.0 ${wrist_1_length} 0.0" rpy="0.0 0.0 -1.5707" />
+      <!-- <origin xyz="0.0 ${wrist_1_length} 0.0" rpy="0.0 0.0 0.0" /> -->
       <axis xyz="0 0 1" />
       <xacro:unless value="${joint_limited}">
@@ -247,4 +252,5 @@
       <child link = "${prefix}wrist_3_link" />
       <origin xyz="0.0 0.0 ${wrist_2_length}" rpy="0.0 0.0 0.0" />
+      <!-- <origin xyz="0.0 0.0 ${wrist_2_length}" rpy="0.0 0.0 0.0" /> -->
       <axis xyz="0 1 0" />
       <xacro:unless value="${joint_limited}">

Commit message: Moved arm to stow position for starting

File: universal_robot/ur_description/urdf/ur5.urdf.xacro (robot description, xacro)
@@ -124,7 +124,7 @@
       <child link = "${prefix}upper_arm_link" />
       <!-- Test arm forward -->
-      <origin xyz="0.0 ${shoulder_offset} 0.0" rpy="0.0 ${pi / 4} 0.0" />
+      <!-- <origin xyz="0.0 ${shoulder_offset} 0.0" rpy="0.0 ${pi / 4} 0.0" /> -->
       <!-- Stow position flat -->
-      <!-- <origin xyz="0.0 ${shoulder_offset} 0.0" rpy="0.0 -1.5707 0.0" /> -->
+      <origin xyz="0.0 ${shoulder_offset} 0.0" rpy="0.0 -1.5707 0.0" />
       <!-- Stow position up -->
       <!-- <origin xyz="0.0 ${shoulder_offset} 0.0" rpy="0.0 -1.122 0.0" /> -->
@@ -160,7 +160,7 @@
       <child link = "${prefix}forearm_link" />
       <!-- Test arm forward -->
-      <origin xyz="0.0 ${elbow_offset} ${upper_arm_length}" rpy="0.0 ${pi / 4} 0.0" />
-      <!-- Stow position up -->
-      <!-- <origin xyz="0.0 ${elbow_offset} ${upper_arm_length}" rpy="0.0 2.6927 0.0" /> -->
+      <!-- <origin xyz="0.0 ${elbow_offset} ${upper_arm_length}" rpy="0.0 ${pi / 4} 0.0" /> -->
+      <!-- Stow position -->
+      <origin xyz="0.0 ${elbow_offset} ${upper_arm_length}" rpy="0.0 2.6927 0.0" />
       <axis xyz="0 1 0" />
       <xacro:unless value="${joint_limited}">
@@ -194,7 +194,7 @@
       <child link = "${prefix}wrist_1_link" />
       <!-- Test arm forward -->
-      <origin xyz="0.0 0.0 ${forearm_length}" rpy="0.0 -1.5707 0.0" />
-      <!-- Stow position down -->
-      <!-- <origin xyz="0.0 0.0 ${forearm_length}" rpy="0.0 -1.122 0.0" /> -->
+      <!-- <origin xyz="0.0 0.0 ${forearm_length}" rpy="0.0 -1.5707 0.0" /> -->
+      <!-- Stow position flat -->
+      <origin xyz="0.0 0.0 ${forearm_length}" rpy="0.0 -1.122 0.0" />
       <!-- Stow position up -->
       <!-- <origin xyz="0.0 0.0 ${forearm_length}" rpy="0.0 -1.5707 0.0" /> -->

Commit message: Put arm in original stow positionw

File: universal_robot/ur_description/urdf/ur5.urdf.xacro (robot description, xacro)
@@ -126,7 +126,7 @@
       <!-- <origin xyz="0.0 ${shoulder_offset} 0.0" rpy="0.0 ${pi / 4} 0.0" /> -->
       <!-- Stow position flat -->
-      <origin xyz="0.0 ${shoulder_offset} 0.0" rpy="0.0 -1.5707 0.0" />
+      <!-- <origin xyz="0.0 ${shoulder_offset} 0.0" rpy="0.0 -1.5707 0.0" /> -->
       <!-- Stow position up -->
-      <!-- <origin xyz="0.0 ${shoulder_offset} 0.0" rpy="0.0 -1.122 0.0" /> -->
+      <origin xyz="0.0 ${shoulder_offset} 0.0" rpy="0.0 -1.122 0.0" />
       <axis xyz="0 1 0" />
       <xacro:unless value="${joint_limited}">
@@ -196,7 +196,7 @@
       <!-- <origin xyz="0.0 0.0 ${forearm_length}" rpy="0.0 -1.5707 0.0" /> -->
       <!-- Stow position flat -->
-      <origin xyz="0.0 0.0 ${forearm_length}" rpy="0.0 -1.122 0.0" />
+      <!-- <origin xyz="0.0 0.0 ${forearm_length}" rpy="0.0 -1.122 0.0" /> -->
       <!-- Stow position up -->
-      <!-- <origin xyz="0.0 0.0 ${forearm_length}" rpy="0.0 -1.5707 0.0" /> -->
+      <origin xyz="0.0 0.0 ${forearm_length}" rpy="0.0 -1.5707 0.0" />
       <axis xyz="0 1 0" />
       <xacro:unless value="${joint_limited}">

Commit message: Added gripper to ur5.urdf.xacro

File: universal_robot/ur_description/urdf/ur5.urdf.xacro (robot description, xacro)
@@ -3,4 +3,5 @@
   <xacro:include filename="$(find ur_description)/urdf/ur.transmission.xacro" />
   <xacro:include filename="$(find ur_description)/urdf/ur.gazebo.xacro" />
+  <xacro:include filename="$(find gripper_description)/urdf/gripper.urdf.xacro" />
   <property name="pi" value="3.14159265" />
   <property name="stl_scale" value="0.001" />
@@ -388,4 +389,11 @@
        </link>
     </xacro:if>
+    <xacro:if value="$(arg ur5_mbzirc_gripper_enabled)">
+      <joint name="${prefix}gripper_wrist_3_link_gripper_base_link_joint" type="fixed">
+        <origin xyz="0.0 ${wrist_3_length} 0.0" rpy="0.0 0.0 0.0" />
+        <parent link="${prefix}wrist_3_link" />
+        <child link="${prefix}gripper_base_link" />
+      </joint>
+    </xacro:if>
   </xacro:macro>
 </robot>

Commit message: Update ur5.urdf.xacro

File: universal_robot/ur_description/urdf/ur5.urdf.xacro (robot description, xacro)
@@ -92,6 +92,5 @@
       <parent link="${prefix}base_link" />
       <child link = "${prefix}shoulder_link" />
-      <origin xyz="0.0 0.0 ${shoulder_height}" rpy="0.0 0.0 1.5707" />
-      <!-- <origin xyz="0.0 0.0 ${shoulder_height}" rpy="0.0 0.0 0.0" /> -->
+      <origin xyz="0.0 0.0 ${shoulder_height}" rpy="0.0 0.0 0.0" />
       <axis xyz="0 0 1" />
       <xacro:unless value="${joint_limited}">
@@ -124,10 +123,5 @@
       <parent link="${prefix}shoulder_link" />
       <child link = "${prefix}upper_arm_link" />
-      <!-- Test arm forward -->
-      <!-- <origin xyz="0.0 ${shoulder_offset} 0.0" rpy="0.0 ${pi / 4} 0.0" /> -->
-      <!-- Stow position flat -->
-      <!-- <origin xyz="0.0 ${shoulder_offset} 0.0" rpy="0.0 -1.5707 0.0" /> -->
-      <!-- Stow position up -->
-      <origin xyz="0.0 ${shoulder_offset} 0.0" rpy="0.0 -1.122 0.0" />
+      <origin xyz="0.0 ${shoulder_offset} 0.0" rpy="0.0 ${pi / 2.0} 0.0" />
       <axis xyz="0 1 0" />
       <xacro:unless value="${joint_limited}">
@@ -160,8 +154,5 @@
       <parent link="${prefix}upper_arm_link" />
       <child link = "${prefix}forearm_link" />
-      <!-- Test arm forward -->
-      <!-- <origin xyz="0.0 ${elbow_offset} ${upper_arm_length}" rpy="0.0 ${pi / 4} 0.0" /> -->
-      <!-- Stow position -->
-      <origin xyz="0.0 ${elbow_offset} ${upper_arm_length}" rpy="0.0 2.6927 0.0" />
+      <origin xyz="0.0 ${elbow_offset} ${upper_arm_length}" rpy="0.0 0.0 0.0" />
       <axis xyz="0 1 0" />
       <xacro:unless value="${joint_limited}">
@@ -194,10 +185,5 @@
       <parent link="${prefix}forearm_link" />
       <child link = "${prefix}wrist_1_link" />
-      <!-- Test arm forward -->
-      <!-- <origin xyz="0.0 0.0 ${forearm_length}" rpy="0.0 -1.5707 0.0" /> -->
-      <!-- Stow position flat -->
-      <!-- <origin xyz="0.0 0.0 ${forearm_length}" rpy="0.0 -1.122 0.0" /> -->
-      <!-- Stow position up -->
-      <origin xyz="0.0 0.0 ${forearm_length}" rpy="0.0 -1.5707 0.0" />
+      <origin xyz="0.0 0.0 ${forearm_length}" rpy="0.0 ${pi / 2.0} 0.0" />
       <axis xyz="0 1 0" />
       <xacro:unless value="${joint_limited}">
@@ -230,6 +216,5 @@
       <parent link="${prefix}wrist_1_link" />
       <child link = "${prefix}wrist_2_link" />
-      <origin xyz="0.0 ${wrist_1_length} 0.0" rpy="0.0 0.0 -1.5707" />
-      <!-- <origin xyz="0.0 ${wrist_1_length} 0.0" rpy="0.0 0.0 0.0" /> -->
+      <origin xyz="0.0 ${wrist_1_length} 0.0" rpy="0.0 0.0 0.0" />
       <axis xyz="0 0 1" />
       <xacro:unless value="${joint_limited}">
@@ -263,5 +248,4 @@
       <child link = "${prefix}wrist_3_link" />
       <origin xyz="0.0 0.0 ${wrist_2_length}" rpy="0.0 0.0 0.0" />
-      <!-- <origin xyz="0.0 0.0 ${wrist_2_length}" rpy="0.0 0.0 0.0" /> -->
       <axis xyz="0 1 0" />
       <xacro:unless value="${joint_limited}">
@@ -397,3 +381,3 @@
     </xacro:if>
   </xacro:macro>
-</robot>
+  </robot>

Commit message: Reverted ur5.urdf.xacro to original angles

File: universal_robot/ur_description/urdf/ur5.urdf.xacro (robot description, xacro)
@@ -92,6 +92,5 @@
       <parent link="${prefix}base_link" />
       <child link = "${prefix}shoulder_link" />
-      <origin xyz="0.0 0.0 ${shoulder_height}" rpy="0.0 0.0 1.5707" />
-      <!-- <origin xyz="0.0 0.0 ${shoulder_height}" rpy="0.0 0.0 0.0" /> -->
+      <origin xyz="0.0 0.0 ${shoulder_height}" rpy="0.0 0.0 0.0" />
       <axis xyz="0 0 1" />
       <xacro:unless value="${joint_limited}">
@@ -124,10 +123,5 @@
       <parent link="${prefix}shoulder_link" />
       <child link = "${prefix}upper_arm_link" />
-      <!-- Test arm forward -->
-      <!-- <origin xyz="0.0 ${shoulder_offset} 0.0" rpy="0.0 ${pi / 4} 0.0" /> -->
-      <!-- Stow position flat -->
-      <!-- <origin xyz="0.0 ${shoulder_offset} 0.0" rpy="0.0 -1.5707 0.0" /> -->
-      <!-- Stow position up -->
-      <origin xyz="0.0 ${shoulder_offset} 0.0" rpy="0.0 -1.122 0.0" />
+      <origin xyz="0.0 ${shoulder_offset} 0.0" rpy="0.0 ${pi / 2.0} 0.0" />
       <axis xyz="0 1 0" />
       <xacro:unless value="${joint_limited}">
@@ -160,8 +154,5 @@
       <parent link="${prefix}upper_arm_link" />
       <child link = "${prefix}forearm_link" />
-      <!-- Test arm forward -->
-      <!-- <origin xyz="0.0 ${elbow_offset} ${upper_arm_length}" rpy="0.0 ${pi / 4} 0.0" /> -->
-      <!-- Stow position -->
-      <origin xyz="0.0 ${elbow_offset} ${upper_arm_length}" rpy="0.0 2.6927 0.0" />
+      <origin xyz="0.0 ${elbow_offset} ${upper_arm_length}" rpy="0.0 0.0 0.0" />
       <axis xyz="0 1 0" />
       <xacro:unless value="${joint_limited}">
@@ -194,10 +185,5 @@
       <parent link="${prefix}forearm_link" />
       <child link = "${prefix}wrist_1_link" />
-      <!-- Test arm forward -->
-      <!-- <origin xyz="0.0 0.0 ${forearm_length}" rpy="0.0 -1.5707 0.0" /> -->
-      <!-- Stow position flat -->
-      <!-- <origin xyz="0.0 0.0 ${forearm_length}" rpy="0.0 -1.122 0.0" /> -->
-      <!-- Stow position up -->
-      <origin xyz="0.0 0.0 ${forearm_length}" rpy="0.0 -1.5707 0.0" />
+      <origin xyz="0.0 0.0 ${forearm_length}" rpy="0.0 ${pi / 2.0} 0.0" />
       <axis xyz="0 1 0" />
       <xacro:unless value="${joint_limited}">
@@ -230,6 +216,5 @@
       <parent link="${prefix}wrist_1_link" />
       <child link = "${prefix}wrist_2_link" />
-      <origin xyz="0.0 ${wrist_1_length} 0.0" rpy="0.0 0.0 -1.5707" />
-      <!-- <origin xyz="0.0 ${wrist_1_length} 0.0" rpy="0.0 0.0 0.0" /> -->
+      <origin xyz="0.0 ${wrist_1_length} 0.0" rpy="0.0 0.0 0.0" />
       <axis xyz="0 0 1" />
       <xacro:unless value="${joint_limited}">
@@ -263,5 +248,4 @@
       <child link = "${prefix}wrist_3_link" />
       <origin xyz="0.0 0.0 ${wrist_2_length}" rpy="0.0 0.0 0.0" />
-      <!-- <origin xyz="0.0 0.0 ${wrist_2_length}" rpy="0.0 0.0 0.0" /> -->
       <axis xyz="0 1 0" />
       <xacro:unless value="${joint_limited}">
