Commit message: Minor formatting changes.  Robot balancing and arm stowing

File: gripper/mybot_description/urdf/gripper.xacro (robot description, xacro)
@@ -30,5 +30,5 @@
 <xacro:property name="chassisLength" value="0.15"/>
 <xacro:property name="chassisWidth" value="0.1"/>
-<xacro:property name="chassisMass" value="50"/>
+<xacro:property name="chassisMass" value="0"/>
 <xacro:property name="casterRadius" value="0.025"/>
 <xacro:property name="casterMass" value="2.5"/>

File: husky/husky_description/urdf/husky.urdf.xacro (robot description, xacro)
@@ -76,6 +76,9 @@
     <link name="inertial_link">
       <inertial>
+        <!-- <mass value="33.455" /> -->
         <mass value="60" />
+        <!-- <origin xyz="-0.08748 -0.00085 -0.2" /> -->
         <origin xyz="-0.08748 -0.00085 0.09947" />
+        <!-- <inertia ixx="1.0" ixy="0.0" ixz="0.0" iyy="1.0" iyz="0.0" izz="1.0" /> -->
         <inertia ixx="1.08995475113" ixy="-0.0427873303" ixz="-0.2166515837" iyy="3.14678733031" iyz="-0.00279457012" izz="3.67348416289" />
       </inertial>

File: universal_robot/ur_description/urdf/ur5.urdf.xacro (robot description, xacro)
@@ -123,6 +123,10 @@
       <parent link="${prefix}shoulder_link" />
       <child link = "${prefix}upper_arm_link" />
-      <origin xyz="0.0 ${shoulder_offset} 0.0" rpy="0.0 -1.122 0.0" />
-      <!-- <origin xyz="0.0 ${shoulder_offset} 0.0" rpy="0.0 ${pi / 2.0} 0.0" /> -->
+      <!-- Test arm forward -->
+      <origin xyz="0.0 ${shoulder_offset} 0.0" rpy="0.0 ${pi / 4} 0.0" />
+      <!-- Stow position flat -->
+      <!-- <origin xyz="0.0 ${shoulder_offset} 0.0" rpy="0.0 -1.5707 0.0" /> -->
+      <!-- Stow position up -->
+      <!-- <origin xyz="0.0 ${shoulder_offset} 0.0" rpy="0.0 -1.122 0.0" /> -->
       <axis xyz="0 1 0" />
       <xacro:unless value="${joint_limited}">
@@ -155,6 +159,8 @@
       <parent link="${prefix}upper_arm_link" />
       <child link = "${prefix}forearm_link" />
-      <origin xyz="0.0 ${elbow_offset} ${upper_arm_length}" rpy="0.0 2.6927 0.0" />
-      <!-- <origin xyz="0.0 ${elbow_offset} ${upper_arm_length}" rpy="0.0 0.0 0.0" /> -->
+      <!-- Test arm forward -->
+      <origin xyz="0.0 ${elbow_offset} ${upper_arm_length}" rpy="0.0 ${pi / 4} 0.0" />
+      <!-- Stow position up -->
+      <!-- <origin xyz="0.0 ${elbow_offset} ${upper_arm_length}" rpy="0.0 2.6927 0.0" /> -->
       <axis xyz="0 1 0" />
       <xacro:unless value="${joint_limited}">
@@ -187,6 +193,10 @@
       <parent link="${prefix}forearm_link" />
       <child link = "${prefix}wrist_1_link" />
+      <!-- Test arm forward -->
       <origin xyz="0.0 0.0 ${forearm_length}" rpy="0.0 -1.5707 0.0" />
-      <!-- <origin xyz="0.0 0.0 ${forearm_length}" rpy="0.0 ${pi / 2.0} 0.0" /> -->
+      <!-- Stow position down -->
+      <!-- <origin xyz="0.0 0.0 ${forearm_length}" rpy="0.0 -1.122 0.0" /> -->
+      <!-- Stow position up -->
+      <!-- <origin xyz="0.0 0.0 ${forearm_length}" rpy="0.0 -1.5707 0.0" /> -->
       <axis xyz="0 1 0" />
       <xacro:unless value="${joint_limited}">

Commit message: modifications made to include the motor and the camera into the URDF of the gripper

File: gripper/mybot_description/urdf/gripper.xacro (robot description, xacro)
@@ -45,5 +45,5 @@
 <xacro:property name="link1Length" value="0.2"/>
 <xacro:property name="link1Width" value="0.02"/>
-<xacro:property name="link1Mass" value="2.9"/>
+<xacro:property name="link1Mass" value="3.5"/>
 <xacro:property name="link2Height" value="0.12"/>
 <xacro:property name="link2Length" value="0.02"/>
@@ -63,5 +63,5 @@
     <origin xyz="0 0 0" rpy="0 0 0"/>
     <geometry>
-      <mesh filename="package://mybot_description/meshes/link1.DAE"/>
+      <mesh filename="package://mybot_description/meshes/gripper_assem.STL"/>
     </geometry>
   </collision>
@@ -69,5 +69,5 @@
    <origin xyz="0 0 0" rpy="0 0 0"/>
     <geometry>
-<mesh filename="package://mybot_description/meshes/link1.DAE"/>
+<mesh filename="package://mybot_description/meshes/gripper_assem.STL"/>
     </geometry>
     <material name="white"/>
@@ -84,5 +84,5 @@
   <child link="link2"/>
 </joint>
-<link name='link2'>
+<!--link name='link2'>
   <collision>
     <origin xyz="0 0 0" rpy="0 0 ${PI}"/>
@@ -103,5 +103,5 @@
     <box_inertia m="${link2Mass}" x="${link2Length}" y="${link2Width}" z="${link2Height}"/>
   </inertial>
-</link>
+</link-->
 <joint name="left_tip_hinge" type="revolute">
   <parent link="link2"/>

File: gripper/mybot_description/urdf/mybot.xacro (robot description, xacro)
@@ -93,5 +93,5 @@
 <link name='base'>
   <collision>
-    <origin xyz="0 0 0" rpy="0 0 0"/>
+    <origin xyz="0 -0.012 -0.063" rpy="0 0 ${PI/2}"/>
     <geometry>
       <mesh filename="package://mybot_description/meshes/base.DAE"/>
@@ -99,5 +99,5 @@
   </collision>
   <visual>
-  <origin xyz="0 0 0" rpy="0 0 0"/>
+  <origin xyz="0 -0.012 -0.063" rpy="0 0 ${PI/2}"/>
     <geometry>
 <mesh filename="package://mybot_description/meshes/base.DAE"/>
@@ -120,5 +120,5 @@
     <origin xyz="0 0 0" rpy="0 0 0"/>
     <geometry>
-      <mesh filename="package://mybot_description/meshes/link1.DAE"/>
+     <mesh filename="package://mybot_description/meshes/link1.DAE"/>
     </geometry>
   </collision>
@@ -126,5 +126,5 @@
    <origin xyz="0 0 0" rpy="0 0 0"/>
     <geometry>
-<mesh filename="package://mybot_description/meshes/link1.DAE"/>
+     <mesh filename="package://mybot_description/meshes/link1.DAE"/>
     </geometry>
     <material name="white"/>

Commit message: Revert "update gripper installation instruction and the gripper URDF"

File: gripper/mybot_description/urdf/gripper.xacro (robot description, xacro)
@@ -45,5 +45,5 @@
 <xacro:property name="link1Length" value="0.2"/>
 <xacro:property name="link1Width" value="0.02"/>
-<xacro:property name="link1Mass" value="3.5"/>
+<xacro:property name="link1Mass" value="2.9"/>
 <xacro:property name="link2Height" value="0.12"/>
 <xacro:property name="link2Length" value="0.02"/>
@@ -63,5 +63,5 @@
     <origin xyz="0 0 0" rpy="0 0 0"/>
     <geometry>
-      <mesh filename="package://mybot_description/meshes/gripper_assem.STL"/>
+      <mesh filename="package://mybot_description/meshes/link1.DAE"/>
     </geometry>
   </collision>
@@ -69,5 +69,5 @@
    <origin xyz="0 0 0" rpy="0 0 0"/>
     <geometry>
-<mesh filename="package://mybot_description/meshes/gripper_assem.STL"/>
+<mesh filename="package://mybot_description/meshes/link1.DAE"/>
     </geometry>
     <material name="white"/>
@@ -84,5 +84,5 @@
   <child link="link2"/>
 </joint>
-<!--link name='link2'>
+<link name='link2'>
   <collision>
     <origin xyz="0 0 0" rpy="0 0 ${PI}"/>
@@ -103,5 +103,5 @@
     <box_inertia m="${link2Mass}" x="${link2Length}" y="${link2Width}" z="${link2Height}"/>
   </inertial>
-</link-->
+</link>
 <joint name="left_tip_hinge" type="revolute">
   <parent link="link2"/>

File: gripper/mybot_description/urdf/mybot.xacro (robot description, xacro)
@@ -93,5 +93,5 @@
 <link name='base'>
   <collision>
-    <origin xyz="0 -0.012 -0.063" rpy="0 0 ${PI/2}"/>
+    <origin xyz="0 0 0" rpy="0 0 0"/>
     <geometry>
       <mesh filename="package://mybot_description/meshes/base.DAE"/>
@@ -99,5 +99,5 @@
   </collision>
   <visual>
-  <origin xyz="0 -0.012 -0.063" rpy="0 0 ${PI/2}"/>
+  <origin xyz="0 0 0" rpy="0 0 0"/>
     <geometry>
 <mesh filename="package://mybot_description/meshes/base.DAE"/>
@@ -120,5 +120,5 @@
     <origin xyz="0 0 0" rpy="0 0 0"/>
     <geometry>
-     <mesh filename="package://mybot_description/meshes/link1.DAE"/>
+      <mesh filename="package://mybot_description/meshes/link1.DAE"/>
     </geometry>
   </collision>
@@ -126,5 +126,5 @@
    <origin xyz="0 0 0" rpy="0 0 0"/>
     <geometry>
-     <mesh filename="package://mybot_description/meshes/link1.DAE"/>
+<mesh filename="package://mybot_description/meshes/link1.DAE"/>
     </geometry>
     <material name="white"/>

Commit message: Updated URDF

File: gripper/mybot_description/urdf/gripper.xacro (robot description, xacro)
@@ -1,5 +1,5 @@
 <?xml version="1.0"?>
 <robot name="mybot" xmlns:xacro="http://ros.org/wiki/xacro">
-<link name='base'>
+<link name='mbzirc_gripper_base'>
   <collision>
     <origin xyz="0 0 0" rpy="0 0 0"/>
@@ -22,5 +22,5 @@
 </link>
 <joint name="base_to_link1" type="fixed">
-  <parent link="base"/>
+  <parent link="mbzirc_gripper_base"/>
   <child link="link1"/>
  <origin xyz="0 0.005 -0.07" rpy="0 0 ${PI/2}"/>
@@ -162,5 +162,5 @@
 <joint name="base_to_camera" type="fixed">
     <origin xyz="0 0 0" rpy="0 0 ${PI/2}"/>
-  <parent link="base"/>
+  <parent link="mbzirc_gripper_base"/>
   <child link="camera"/>
 </joint>

File: husky/husky_description/urdf/description.xacro (robot description, xacro)
@@ -25,4 +25,5 @@
   <xacro:arg name="ur5_enabled" default="false" />
   <xacro:arg name="ur5_camera_enabled" default="false" />
+  <xacro:arg name="ur5_mbzirc_gripper_enabled" default="false" />
   <xacro:arg name="kinect_enabled" default="false" />
   <xacro:arg name="kinectv2_enabled" default="false" />

File: husky/husky_description/urdf/husky.urdf.xacro (robot description, xacro)
@@ -76,12 +76,9 @@
     <link name="inertial_link">
       <inertial>
-        <!-- <mass value="33.455" /> -->
         <mass value="60" />
-        <!-- <origin xyz="-0.08748 -0.00085 -0.2" /> -->
         <origin xyz="-0.08748 -0.00085 0.09947" />
-        <!-- <inertia ixx="1.0" ixy="0.0" ixz="0.0" iyy="1.0" iyz="0.0" izz="1.0" /> -->
         <inertia ixx="1.08995475113" ixy="-0.0427873303" ixz="-0.2166515837" iyy="3.14678733031" iyz="-0.00279457012" izz="3.67348416289" />
       </inertial>
-</link>
+    </link>
     <joint name="inertial_joint" type="fixed">
       <origin xyz="0 0 0" rpy="0 0 0" />
@@ -123,14 +120,17 @@
         <origin xyz="0.3058 0 0.0065" rpy="0.0 0.0 -1.57079632679" />
       </joint>
-      <!-- Spawn gripper-->
-      <xacro:gripper />
-      <!-- Join Gripper -->
-        <joint name="base_to_arm" type="fixed">
-          <parent link="ur5_arm_wrist_3_link"/>
-          <child link="base"/>
-          <origin xyz="0 0.09 0" rpy="0 0 0"/>
-        </joint>
     </xacro:if>
     <xacro:if value="$(arg ur5_camera_enabled)">
+      <xacro:property name="reflect" value="-1" />
+      <!-- Spawn arm -->
+      <xacro:ur5_robot prefix="ur5_arm_" joint_limited="true"/>
+      <!-- Join arm -->
+      <joint name="ur5_arm_base" type="fixed">
+        <parent link="top_plate_link" />
+        <child link="ur5_arm_base_link" />
+        <origin xyz="0.3058 0 0.0065" rpy="0.0 0.0 -1.57079632679" />
+      </joint>
+    </xacro:if>
+    <xacro:if value="$(arg ur5_mbzirc_gripper_enabled)">
       <xacro:property name="reflect" value="-1" />
       <!-- Spawn arm -->

File: universal_robot/ur_description/urdf/ur5.urdf.xacro (robot description, xacro)
@@ -3,4 +3,5 @@
   <xacro:include filename="$(find ur_description)/urdf/ur.transmission.xacro" />
   <xacro:include filename="$(find ur_description)/urdf/ur.gazebo.xacro" />
+  <xacro:include filename="$(find mybot_description)/urdf/gripper.xacro" />
   <property name="pi" value="3.14159265" />
   <property name="stl_scale" value="0.001" />
@@ -388,4 +389,11 @@
        </link>
     </xacro:if>
+    <xacro:if value="$(arg ur5_mbzirc_gripper_enabled)">
+      <joint name="${prefix}mbzirc_gripper_joint" type="fixed">
+        <origin xyz="0.0 ${wrist_3_length} 0.0" rpy="0.0 0.0 0.0" />
+        <parent link="${prefix}wrist_3_link" />
+        <child link="mbzirc_gripper_base" />
+      </joint>
+    </xacro:if>
   </xacro:macro>
 </robot>
