Commit message: Changed gripper to a xacro and updated ur5.urdf.xacro

File: gripper/mybot_description/urdf/gripper.xacro (robot description, xacro)
@@ -1,207 +1,209 @@
 <?xml version="1.0"?>
-<robot name="mybot" xmlns:xacro="http://ros.org/wiki/xacro">
-<link name='mbzirc_gripper_base'>
-  <collision>
-    <origin xyz="0 0 0" rpy="0 0 0"/>
-    <geometry>
-      <mesh filename="package://mybot_description/meshes/base.DAE"/>
-    </geometry>
-  </collision>
-  <visual>
-  <origin xyz="0 0 0" rpy="0 0 0"/>
-    <geometry>
-<mesh filename="package://mybot_description/meshes/base.DAE"/>
-    </geometry>
-    <material name="white"/>
-  </visual>
-  <inertial>
-    <origin xyz="0 0 0" rpy="0 0 0"/>
-    <mass value="${baseMass}"/>
-    <box_inertia m="${baseMass}" x="${baseLength}" y="${baseWidth}" z="${baseHeight}"/>
-  </inertial>
-</link>
-<joint name="base_to_link1" type="fixed">
-  <parent link="mbzirc_gripper_base"/>
-  <child link="link1"/>
- <origin xyz="0 0.005 -0.07" rpy="0 0 ${PI/2}"/>
-</joint>
-<xacro:property name="PI" value="3.1415926535897931"/>
-<xacro:property name="chassisHeight" value="0.05"/>
-<xacro:property name="chassisLength" value="0.15"/>
-<xacro:property name="chassisWidth" value="0.1"/>
-<xacro:property name="chassisMass" value="0"/>
-<xacro:property name="casterRadius" value="0.025"/>
-<xacro:property name="casterMass" value="2.5"/>
-<xacro:property name="wheelWidth" value="0.025"/>
-<xacro:property name="wheelRadius" value="0.05"/>
-<xacro:property name="wheelPos" value="-0.15"/>
-<xacro:property name="wheelMass" value="2.5"/>
-<xacro:property name="EndEffectorHeight" value="0.55"/>
-<xacro:property name="baseHeight" value="0.15"/>
-<xacro:property name="baseLength" value="0.01"/>
-<xacro:property name="baseWidth" value="0.08"/>
-<xacro:property name="baseMass" value="2.7"/>
-<xacro:property name="link1Height" value="0.1"/>
-<xacro:property name="link1Length" value="0.2"/>
-<xacro:property name="link1Width" value="0.02"/>
-<xacro:property name="link1Mass" value="2.9"/>
-<xacro:property name="link2Height" value="0.12"/>
-<xacro:property name="link2Length" value="0.02"/>
-<xacro:property name="link2Width" value="0.02"/>
-<xacro:property name="link2Mass" value="2.2"/>
-<xacro:property name="tipHeight" value="0.3"/>
-<xacro:property name="tipLength" value="0.05"/>
-<xacro:property name="tipWidth" value="0.03"/>
-<xacro:property name="tipMass" value="2.07"/>
-<xacro:property name="cameraSize" value="0.025"/>
-<xacro:property name="cameraMass" value="0.05"/>
- <xacro:include filename="$(find mybot_description)/urdf/gripper.gazebo" />
- <xacro:include filename="$(find mybot_description)/urdf/materials.xacro" />
- <xacro:include filename="$(find mybot_description)/urdf/macros.xacro" />
-<link name='link1'>
-  <collision>
-    <origin xyz="0 0 0" rpy="0 0 0"/>
-    <geometry>
-      <mesh filename="package://mybot_description/meshes/link1.DAE"/>
-    </geometry>
-  </collision>
-  <visual>
-   <origin xyz="0 0 0" rpy="0 0 0"/>
-    <geometry>
-<mesh filename="package://mybot_description/meshes/link1.DAE"/>
-    </geometry>
-    <material name="white"/>
-  </visual>
-  <inertial>
-     <origin xyz="0 0 0" rpy="0 0 0"/>
-    <mass value="${link1Mass}"/>
-    <box_inertia m="${link1Mass}" x="${link1Length}" y="${link1Width}" z="${link1Height}"/>
-  </inertial>
-</link>
-<joint name="link1_to_link2" type="fixed">
-    <origin xyz="0.104 0 0" rpy="0 0 ${PI/2}"/>
-  <parent link="link1"/>
-  <child link="link2"/>
-</joint>
-<link name='link2'>
-  <collision>
-    <origin xyz="0 0 0" rpy="0 0 ${PI}"/>
-    <geometry>
-      <mesh filename="package://mybot_description/meshes/link2.DAE"/>
-    </geometry>
-  </collision>
-  <visual>
-    <origin xyz="0 0 0" rpy="0 0 ${PI}"/>
-    <geometry>
-<mesh filename="package://mybot_description/meshes/link2.DAE"/>
-    </geometry>
-    <material name="white"/>
-  </visual>
-  <inertial>
-    <origin xyz="0 0 0" rpy="0 0 0"/>
-    <mass value="${link2Mass}"/>
-    <box_inertia m="${link2Mass}" x="${link2Length}" y="${link2Width}" z="${link2Height}"/>
-  </inertial>
-</link>
-<joint name="left_tip_hinge" type="revolute">
-  <parent link="link2"/>
-  <child link="left_tip"/>
-<origin xyz="0.0125 0 0.00025" rpy="0 0 -${PI/2}" />
-  <axis xyz="0 0 1" rpy="0 0 0" />
-  <limit effort="100" velocity="5" lower="-0.037" upper="0.6" />
-  <joint_properties damping="0.0" friction="10.0"/>
-</joint>
-<link name='left_tip'>
-  <collision>
-   <origin xyz="0 0 0" rpy="0 0 0" />
-    <geometry>
-      <mesh filename="package://mybot_description/meshes/tip.DAE"/>
-    </geometry>
-  </collision>
-  <visual>
-   <origin xyz="0 0 0" rpy="0 0 0" />
-    <geometry>
-<mesh filename="package://mybot_description/meshes/tip.DAE"/>
-    </geometry>
-    <material name="white"/>
-  </visual>
-  <inertial>
-    <origin xyz="0 0 0" rpy="0 0 0"/>
-    <mass value="${tipMass}"/>
-    <box_inertia m="${tipMass}" x="${tipLength}" y="${tipWidth}" z="${tipHeight}"/>
-  </inertial>
-</link>
-<joint name="right_tip_hinge" type="revolute">
-  <parent link="link2"/>
-  <child link="right_tip"/>
-<origin xyz="-0.0125 0 0.00025" rpy="0 0 ${PI/2}" />
-  <axis xyz="0 0 1" rpy="0 0 0" />
-  <limit effort="100" velocity="5" lower="-0.6" upper="0.037" />
-  <joint_properties damping="0.0" friction="10.0"/>
-</joint>
-<link name='right_tip'>
-  <collision>
-   <origin xyz="0 0 0" rpy="0 ${PI} 0" />
-    <geometry>
-      <mesh filename="package://mybot_description/meshes/tip.DAE"/>
-    </geometry>
-  </collision>
-  <visual>
-   <origin xyz="0 0 0" rpy="0 ${PI} 0" />
-    <geometry>
-<mesh filename="package://mybot_description/meshes/tip.DAE"/>
-    </geometry>
-    <material name="white"/>
-  </visual>
-  <inertial>
-    <origin xyz="0 0 0" rpy="0 0 0"/>
-    <mass value="${tipMass}"/>
-    <box_inertia m="${tipMass}" x="${tipLength}" y="${tipWidth}" z="${tipHeight}"/>
-  </inertial>
-</link>
-<joint name="base_to_camera" type="fixed">
-    <origin xyz="0 0 0" rpy="0 0 ${PI/2}"/>
-  <parent link="mbzirc_gripper_base"/>
-  <child link="camera"/>
-</joint>
-<link name="camera">
-  <collision>
-    <origin xyz="0 0 0" rpy="0 0 0"/>
-    <geometry>
-      <box size="${cameraSize*2} ${cameraSize/2} ${cameraSize/2}"/>
-    </geometry>
-  </collision>
-  <visual>
-   <origin xyz="0 0 0" rpy="0 0 0"/>
-    <geometry>
-      <box size="${cameraSize*2} ${cameraSize} ${cameraSize/2}"/>
-    </geometry>
-    <material name="black"/>
-  </visual>
-  <inertial>
-    <mass value="${cameraMass}" />
-    <origin xyz="0 0 0" rpy="0 0 0"/>
-    <box_inertia m="${cameraMass}" x="${cameraSize*2}" y="${cameraSize}" z="${cameraSize/2}" />
-  </inertial>
-</link>
-<transmission name="left_trans">
-  <type>transmission_interface/SimpleTransmission</type>
-  <joint name="left_tip_hinge">
-    <hardwareInterface>EffortJointInterface</hardwareInterface>
- </joint>
-  <actuator name="$left_Motor">
-    <hardwareInterface>EffortJointInterface</hardwareInterface>
-    <mechanicalReduction>1</mechanicalReduction>
-  </actuator>
-</transmission>
-<transmission name="right_trans">
-  <type>transmission_interface/SimpleTransmission</type>
-  <joint name="right_tip_hinge">
-    <hardwareInterface>EffortJointInterface</hardwareInterface>
- </joint>
-  <actuator name="$right_Motor">
-    <hardwareInterface>EffortJointInterface</hardwareInterface>
-    <mechanicalReduction>1</mechanicalReduction>
-  </actuator>
-</transmission>
+<robot xmlns:xacro="http://www.ros.org/wiki/xacro">
+  <xacro:property name="PI" value="3.1415926535897931"/>
+  <xacro:property name="chassisHeight" value="0.05"/>
+  <xacro:property name="chassisLength" value="0.15"/>
+  <xacro:property name="chassisWidth" value="0.1"/>
+  <xacro:property name="chassisMass" value="0"/>
+  <xacro:property name="casterRadius" value="0.025"/>
+  <xacro:property name="casterMass" value="2.5"/>
+  <xacro:property name="wheelWidth" value="0.025"/>
+  <xacro:property name="wheelRadius" value="0.05"/>
+  <xacro:property name="wheelPos" value="-0.15"/>
+  <xacro:property name="wheelMass" value="2.5"/>
+  <xacro:property name="EndEffectorHeight" value="0.55"/>
+  <xacro:property name="baseHeight" value="0.15"/>
+  <xacro:property name="baseLength" value="0.01"/>
+  <xacro:property name="baseWidth" value="0.08"/>
+  <xacro:property name="baseMass" value="2.7"/>
+  <xacro:property name="link1Height" value="0.1"/>
+  <xacro:property name="link1Length" value="0.2"/>
+  <xacro:property name="link1Width" value="0.02"/>
+  <xacro:property name="link1Mass" value="2.9"/>
+  <xacro:property name="link2Height" value="0.12"/>
+  <xacro:property name="link2Length" value="0.02"/>
+  <xacro:property name="link2Width" value="0.02"/>
+  <xacro:property name="link2Mass" value="2.2"/>
+  <xacro:property name="tipHeight" value="0.3"/>
+  <xacro:property name="tipLength" value="0.05"/>
+  <xacro:property name="tipWidth" value="0.03"/>
+  <xacro:property name="tipMass" value="2.07"/>
+  <xacro:property name="cameraSize" value="0.025"/>
+  <xacro:property name="cameraMass" value="0.05"/>
+  <xacro:include filename="$(find mybot_description)/urdf/gripper.gazebo" />
+  <xacro:include filename="$(find mybot_description)/urdf/materials.xacro" />
+  <xacro:include filename="$(find mybot_description)/urdf/macros.xacro" />
+  <xacro:macro name="gripper" params="prefix">
+    <link name='${prefix}base_link'>
+       <inertial>
+         <origin xyz="0 0 0" rpy="0 0 0"/>
+         <mass value="${baseMass}"/>
+         <box_inertia m="${baseMass}" x="${baseLength}" y="${baseWidth}" z="${baseHeight}"/>
+       </inertial>
+       <visual>
+         <origin xyz="0 0 0" rpy="0 0 0"/>
+         <geometry>
+           <mesh filename="package://mybot_description/meshes/base_link.dae"/>
+         </geometry>
+         <material name="white"/>
+       </visual>
+       <collision>
+         <origin xyz="0 0 0" rpy="0 0 0"/>
+         <geometry>
+           <mesh filename="package://mybot_description/meshes/base_link.stl"/>
+         </geometry>
+       </collision>
+     </link>
+     <joint name="${prefix}base_link_link_1_joint" type="fixed">
+       <parent link="${prefix}base_link"/>
+       <child link="${prefix}link_1"/>
+       <origin xyz="0 0.005 -0.07" rpy="0 0 ${PI/2}"/>
+     </joint>
+    <link name='${prefix}link_1'>
+      <inertial>
+        <origin xyz="0 0 0" rpy="0 0 0"/>
+        <mass value="${link1Mass}"/>
+        <box_inertia m="${link1Mass}" x="${link1Length}" y="${link1Width}" z="${link1Height}"/>
+      </inertial>
+      <visual>
+       <origin xyz="0 0 0" rpy="0 0 0"/>
+        <geometry>
+          <mesh filename="package://mybot_description/meshes/link_1.dae"/>
+        </geometry>
+        <material name="white"/>
+      </visual>
+      <collision>
+        <origin xyz="0 0 0" rpy="0 0 0"/>
+        <geometry>
+          <mesh filename="package://mybot_description/meshes/link_1.stl"/>
+        </geometry>
+      </collision>
+    </link>
+    <joint name="${prefix}link_1_link_2_joint" type="fixed">
+      <origin xyz="0.104 0 0" rpy="0 0 ${PI/2}"/>
+      <parent link="${prefix}link_1"/>
+      <child link="${prefix}link_2"/>
+    </joint>
+    <link name='${prefix}link_2'>
+      <inertial>
+        <origin xyz="0 0 0" rpy="0 0 0"/>
+        <mass value="${link2Mass}"/>
+        <box_inertia m="${link2Mass}" x="${link2Length}" y="${link2Width}" z="${link2Height}"/>
+      </inertial>
+      <visual>
+        <origin xyz="0 0 0" rpy="0 0 ${PI}"/>
+        <geometry>
+          <mesh filename="package://mybot_description/meshes/link_2.dae"/>
+        </geometry>
+        <material name="white"/>
+      </visual>
+      <collision>
+        <origin xyz="0 0 0" rpy="0 0 ${PI}"/>
+        <geometry>
+          <mesh filename="package://mybot_description/meshes/link_2.stl"/>
+        </geometry>
+      </collision>
+    </link>
+    <joint name="${prefix}link_2_left_tip_joint" type="revolute">
+      <parent link="${prefix}link_2"/>
+      <child link="${prefix}left_tip"/>
+      <origin xyz="0.0125 0 0.00025" rpy="0 0 -${PI/2}" />
+      <axis xyz="0 0 1" rpy="0 0 0" />
+      <limit effort="100" velocity="5" lower="-0.037" upper="0.6" />
+      <joint_properties damping="0.0" friction="10.0"/>
+    </joint>
+    <link name='${prefix}left_tip'>
+      <inertial>
+        <origin xyz="0 0 0" rpy="0 0 0"/>
+        <mass value="${tipMass}"/>
+        <box_inertia m="${tipMass}" x="${tipLength}" y="${tipWidth}" z="${tipHeight}"/>
+      </inertial>
+      <visual>
+        <origin xyz="0 0 0" rpy="0 0 0" />
+        <geometry>
+          <mesh filename="package://mybot_description/meshes/tip.dae"/>
+        </geometry>
+        <material name="white"/>
+      </visual>
+      <collision>
+        <origin xyz="0 0 0" rpy="0 0 0" />
+        <geometry>
+          <mesh filename="package://mybot_description/meshes/tip.stl"/>
+        </geometry>
+      </collision>
+    </link>
+    <joint name="${prefix}link_2_right_tip_joint" type="revolute">
+      <parent link="${prefix}link_2"/>
+      <child link="${prefix}right_tip"/>
+      <origin xyz="-0.0125 0 0.00025" rpy="0 0 ${PI/2}" />
+      <axis xyz="0 0 1" rpy="0 0 0" />
+      <limit effort="100" velocity="5" lower="-0.6" upper="0.037" />
+      <joint_properties damping="0.0" friction="10.0"/>
+    </joint>
+    <link name='${prefix}right_tip'>
+      <inertial>
+        <origin xyz="0 0 0" rpy="0 0 0"/>
+        <mass value="${tipMass}"/>
+        <box_inertia m="${tipMass}" x="${tipLength}" y="${tipWidth}" z="${tipHeight}"/>
+      </inertial>
+      <visual>
+        <origin xyz="0 0 0" rpy="0 ${PI} 0" />
+        <geometry>
+          <mesh filename="package://mybot_description/meshes/tip.dae"/>
+        </geometry>
+        <material name="white"/>
+      </visual>
+      <collision>
+        <origin xyz="0 0 0" rpy="0 ${PI} 0" />
+        <geometry>
+          <mesh filename="package://mybot_description/meshes/tip.stl"/>
+        </geometry>
+      </collision>
+    </link>
+    <joint name="${prefix}base_link_camera_joint" type="fixed">
+      <origin xyz="0 0 0" rpy="0 0 ${PI/2}"/>
+      <parent link="${prefix}base_link"/>
+      <child link="${prefix}camera"/>
+    </joint>
+    <link name="${prefix}camera">
+      <inertial>
+        <mass value="${cameraMass}" />
+        <origin xyz="0 0 0" rpy="0 0 0"/>
+        <box_inertia m="${cameraMass}" x="${cameraSize*2}" y="${cameraSize}" z="${cameraSize/2}" />
+      </inertial>
+      <visual>
+        <origin xyz="0 0 0" rpy="0 0 0"/>
+        <geometry>
+          <box size="${cameraSize*2} ${cameraSize} ${cameraSize/2}"/>
+        </geometry>
+        <material name="black"/>
+      </visual>
+      <collision>
+        <origin xyz="0 0 0" rpy="0 0 0"/>
+        <geometry>
+          <box size="${cameraSize*2} ${cameraSize/2} ${cameraSize/2}"/>
+        </geometry>
+      </collision>
+    </link>
+    <transmission name="left_trans">
+      <type>transmission_interface/SimpleTransmission</type>
+      <joint name="${prefix}link_2_left_tip_joint">
+        <hardwareInterface>EffortJointInterface</hardwareInterface>
+     </joint>
+      <actuator name="$left_Motor">
+        <hardwareInterface>EffortJointInterface</hardwareInterface>
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
File: universal_robot/ur_description/urdf/ur5.urdf.xacro (robot description, xacro)
@@ -390,8 +390,9 @@
     </xacro:if>
     <xacro:if value="$(arg ur5_mbzirc_gripper_enabled)">
-      <joint name="${prefix}mbzirc_gripper_joint" type="fixed">
+      <xacro:gripper prefix="ur5_arm_gripper_"/>
+      <joint name="ur5_arm_gripper_wrist_3_link_base_link_joint" type="fixed">
         <origin xyz="0.0 ${wrist_3_length} 0.0" rpy="0.0 0.0 0.0" />
         <parent link="${prefix}wrist_3_link" />
-        <child link="mbzirc_gripper_base" />
+        <child link="ur5_arm_gripper_base_link" />
       </joint>
     </xacro:if>
