Commit message: Updated gripper.xacro to make the gripper a xacro and creatd static urdf

File: gripper/mybot_description/urdf/gripper.xacro (robot description, xacro)
@@ -2,4 +2,5 @@
 <robot xmlns:xacro="http://www.ros.org/wiki/xacro">
   <xacro:property name="PI" value="3.1415926535897931"/>
+  <xacro:property name="stl_scale" value="0.001" />
   <xacro:property name="chassisHeight" value="0.05"/>
   <xacro:property name="chassisLength" value="0.15"/>
@@ -32,5 +33,4 @@
   <xacro:property name="cameraMass" value="0.05"/>
   <xacro:include filename="$(find mybot_description)/urdf/gripper.gazebo" />
-  <xacro:include filename="$(find mybot_description)/urdf/materials.xacro" />
   <xacro:include filename="$(find mybot_description)/urdf/macros.xacro" />
   <xacro:macro name="gripper" params="prefix">
@@ -44,12 +44,11 @@
          <origin xyz="0 0 0" rpy="0 0 0"/>
          <geometry>
-           <mesh filename="package://mybot_description/meshes/base_link.dae"/>
+           <mesh filename="package://mybot_description/meshes/base_link.dae" scale="${stl_scale} ${stl_scale} ${stl_scale}"/>
          </geometry>
-         <material name="white"/>
        </visual>
        <collision>
          <origin xyz="0 0 0" rpy="0 0 0"/>
          <geometry>
-           <mesh filename="package://mybot_description/meshes/base_link.stl"/>
+           <mesh filename="package://mybot_description/meshes/base_link.stl" scale="${stl_scale} ${stl_scale} ${stl_scale}"/>
          </geometry>
        </collision>
@@ -69,12 +68,11 @@
        <origin xyz="0 0 0" rpy="0 0 0"/>
         <geometry>
-          <mesh filename="package://mybot_description/meshes/link_1.dae"/>
-        </geometry>
-        <material name="white"/>
-      </visual>
-      <collision>
-        <origin xyz="0 0 0" rpy="0 0 0"/>
-        <geometry>
-          <mesh filename="package://mybot_description/meshes/link_1.stl"/>
+          <mesh filename="package://mybot_description/meshes/link_1.dae" scale="${stl_scale} ${stl_scale} ${stl_scale}"/>
+        </geometry>
+      </visual>
+      <collision>
+        <origin xyz="0 0 0" rpy="0 0 0"/>
+        <geometry>
+          <mesh filename="package://mybot_description/meshes/link_1.stl" scale="${stl_scale} ${stl_scale} ${stl_scale}"/>
         </geometry>
       </collision>
@@ -94,12 +92,11 @@
         <origin xyz="0 0 0" rpy="0 0 ${PI}"/>
         <geometry>
-          <mesh filename="package://mybot_description/meshes/link_2.dae"/>
-        </geometry>
-        <material name="white"/>
+          <mesh filename="package://mybot_description/meshes/link_2.dae" scale="${stl_scale} ${stl_scale} ${stl_scale}"/>
+        </geometry>
       </visual>
       <collision>
         <origin xyz="0 0 0" rpy="0 0 ${PI}"/>
         <geometry>
-          <mesh filename="package://mybot_description/meshes/link_2.stl"/>
+          <mesh filename="package://mybot_description/meshes/link_2.stl" scale="${stl_scale} ${stl_scale} ${stl_scale}"/>
         </geometry>
       </collision>
@@ -122,12 +119,11 @@
         <origin xyz="0 0 0" rpy="0 0 0" />
         <geometry>
-          <mesh filename="package://mybot_description/meshes/tip.dae"/>
-        </geometry>
-        <material name="white"/>
+          <mesh filename="package://mybot_description/meshes/tip.dae" scale="${stl_scale} ${stl_scale} ${stl_scale}"/>
+        </geometry>
       </visual>
       <collision>
         <origin xyz="0 0 0" rpy="0 0 0" />
         <geometry>
-          <mesh filename="package://mybot_description/meshes/tip.stl"/>
+          <mesh filename="package://mybot_description/meshes/tip.stl" scale="${stl_scale} ${stl_scale} ${stl_scale}"/>
         </geometry>
       </collision>
@@ -150,12 +146,11 @@
         <origin xyz="0 0 0" rpy="0 ${PI} 0" />
         <geometry>
-          <mesh filename="package://mybot_description/meshes/tip.dae"/>
-        </geometry>
-        <material name="white"/>
+          <mesh filename="package://mybot_description/meshes/tip.dae" scale="${stl_scale} ${stl_scale} ${stl_scale}"/>
+        </geometry>
       </visual>
       <collision>
         <origin xyz="0 0 0" rpy="0 ${PI} 0" />
         <geometry>
-          <mesh filename="package://mybot_description/meshes/tip.stl"/>
+          <mesh filename="package://mybot_description/meshes/tip.stl" scale="${stl_scale} ${stl_scale} ${stl_scale}"/>
         </geometry>
       </collision>
@@ -177,5 +172,4 @@
           <box size="${cameraSize*2} ${cameraSize} ${cameraSize/2}"/>
         </geometry>
-        <material name="black"/>
       </visual>
       <collision>

File: husky/husky_description/urdf/description.xacro (robot description, xacro)
@@ -22,10 +22,10 @@
 -->
 <robot name="husky" xmlns:xacro="http://ros.org/wiki/xacro">
-  <xacro:arg name="laser_enabled" default="false" />
+  <xacro:arg name="laser_enabled" default="true" />
   <xacro:arg name="ur5_enabled" default="false" />
   <xacro:arg name="ur5_camera_enabled" default="false" />
-  <xacro:arg name="ur5_mbzirc_gripper_enabled" default="false" />
+  <xacro:arg name="ur5_mbzirc_gripper_enabled" default="true" />
   <xacro:arg name="kinect_enabled" default="false" />
-  <xacro:arg name="kinectv2_enabled" default="false" />
+  <xacro:arg name="kinectv2_enabled" default="true" />
   <xacro:arg name="primesense_enabled" default="false"/>
   <xacro:include filename="$(find husky_description)/urdf/husky.urdf.xacro" />

File: husky/husky_description/urdf/husky_ur5.urdf (robot description, URDF)
Before this commit: robot husky, 32 links, 31 joints
Links:
- removed link camera_optical_frame
- removed link ur5_arm_camera_link
- removed link ur5_arm_camera_mount_link
- removed link ur5_arm_camera_optical_frame
- removed link ur5_arm_laser_pointer_link
- added link kinect2_link
- added link ur5_arm_gripper_base_link, mass 2.7; collision mesh filename=package://mybot_description/meshes/base_link.stl scale=0.001 0.001 0.001; visual mesh filename=package://mybot_description/meshes/base_link.dae scale=0.001 0.001 0.001
- added link ur5_arm_gripper_camera, mass 0.05; collision box size=0.05 0.0125 0.0125; visual box size=0.05 0.025 0.0125
- added link ur5_arm_gripper_left_tip, mass 2.07; collision mesh filename=package://mybot_description/meshes/tip.stl scale=0.001 0.001 0.001; visual mesh filename=package://mybot_description/meshes/tip.dae scale=0.001 0.001 0.001
- added link ur5_arm_gripper_link_1, mass 2.9; collision mesh filename=package://mybot_description/meshes/link_1.stl scale=0.001 0.001 0.001; visual mesh filename=package://mybot_description/meshes/link_1.dae scale=0.001 0.001 0.001
- added link ur5_arm_gripper_link_2, mass 2.2; collision mesh filename=package://mybot_description/meshes/link_2.stl scale=0.001 0.001 0.001; visual mesh filename=package://mybot_description/meshes/link_2.dae scale=0.001 0.001 0.001
- added link ur5_arm_gripper_right_tip, mass 2.07; collision mesh filename=package://mybot_description/meshes/tip.stl scale=0.001 0.001 0.001; visual mesh filename=package://mybot_description/meshes/tip.dae scale=0.001 0.001 0.001
- link sensor_arch_mount_link: mass 20.0 -> None
Joints:
- removed joint camera_optical_joint
- removed joint kinectv2_frame_joint
- removed joint ur5_arm_camera_joint
- removed joint ur5_arm_camera_mount_joint
- removed joint ur5_arm_camera_optical_joint
- removed joint ur5_arm_laser_pointer_joint
- added joint camera_link_joint: type fixed, parent camera_mount_link, child camera_link, origin xyz=0.028 -0.096 0.112 rpy=0.0 0.0 0.0
- added joint kinect2_link_joint: type fixed, parent camera_link, child kinect2_link, origin xyz=0.0 0.0 0.0 rpy=-1.57079632679 0 -1.57079632679
- added joint ur5_arm_gripper_base_link_camera_joint: type fixed, parent ur5_arm_gripper_base_link, child ur5_arm_gripper_camera, origin xyz=0 0 0 rpy=0 0 1.57079632679
- added joint ur5_arm_gripper_base_link_link_1_joint: type fixed, parent ur5_arm_gripper_base_link, child ur5_arm_gripper_link_1, origin xyz=0 0.005 -0.07 rpy=0 0 1.57079632679
- added joint ur5_arm_gripper_link_1_link_2_joint: type fixed, parent ur5_arm_gripper_link_1, child ur5_arm_gripper_link_2, origin xyz=0.104 0 0 rpy=0 0 1.57079632679
- added joint ur5_arm_gripper_link_2_left_tip_joint: type revolute, parent ur5_arm_gripper_link_2, child ur5_arm_gripper_left_tip, origin xyz=0.0125 0 0.00025 rpy=0 0 -1.57079632679, axis 0 0 1, limit lower=-0.037 upper=0.6 effort=100 velocity=5
- added joint ur5_arm_gripper_link_2_right_tip_joint: type revolute, parent ur5_arm_gripper_link_2, child ur5_arm_gripper_right_tip, origin xyz=-0.0125 0 0.00025 rpy=0 0 1.57079632679, axis 0 0 1, limit lower=-0.6 upper=0.037 effort=100 velocity=5
- added joint ur5_arm_gripper_wrist_3_link_base_link_joint: type fixed, parent ur5_arm_wrist_3_link, child ur5_arm_gripper_base_link, origin xyz=0.0 0.0823 0.0 rpy=0.0 0.0 0.0
- joint base_laser_joint: origin xyz=-0.0352 0 -0.0566 rpy=3.14159 0 0 -> xyz=-0.0352 0 -0.0566 rpy=0 0 0
- joint camera_mount_joint: origin xyz=0.0 0.0 0.0 rpy=0.0 0.0 0.0 -> xyz=0.0 0.0 0.0 rpy=0.0 0.0 3.14159265359
- joint imu_joint: origin xyz=0.19 0 0.149 rpy=0 -1.5708 3.14159265359 -> xyz=0.19 0 0.149 rpy=0 -1.57079632679 3.14159265359
- joint ur5_arm_base: origin xyz=0.3058 0 0.0065 rpy=0.0 0.0 -1.57 -> xyz=0.3058 0 0.0065 rpy=0.0 0.0 -1.57079632679
- joint ur5_arm_elbow_joint: origin xyz=0.0 -0.1197 0.425 rpy=0.0 0.0 0.0 -> xyz=0.0 -0.1197 0.425 rpy=0.0 2.6927 0.0
- joint ur5_arm_shoulder_lift_joint: origin xyz=0.0 0.13585 0.0 rpy=0.0 1.570796325 0.0 -> xyz=0.0 0.13585 0.0 rpy=0.0 -1.122 0.0
- joint ur5_arm_shoulder_pan_joint: origin xyz=0.0 0.0 0.089159 rpy=0.0 0.0 0.0 -> xyz=0.0 0.0 0.089159 rpy=0.0 0.0 1.5707
- joint ur5_arm_wrist_1_joint: origin xyz=0.0 0.0 0.39225 rpy=0.0 1.570796325 0.0 -> xyz=0.0 0.0 0.39225 rpy=0.0 -1.5707 0.0
- joint ur5_arm_wrist_2_joint: origin xyz=0.0 0.093 0.0 rpy=0.0 0.0 0.0 -> xyz=0.0 0.093 0.0 rpy=0.0 0.0 -1.5707

File: husky/husky_simulator/husky_gazebo/urdf/husky.gazebo.xacro (robot description, xacro)
@@ -141,5 +141,20 @@
         <selfCollide>true</selfCollide>
       </gazebo>
-      <gazebo reference="mbzirc_gripper_base">
+      <gazebo reference="ur5_arm_gripper_base_link">
+        <selfCollide>true</selfCollide>
+      </gazebo>
+      <gazebo reference="ur5_arm_gripper_camera">
+        <selfCollide>true</selfCollide>
+      </gazebo>
+      <gazebo reference="ur5_arm_gripper_link_1">
+        <selfCollide>true</selfCollide>
+      </gazebo>
+      <gazebo reference="ur5_arm_gripper_link_2">
+        <selfCollide>true</selfCollide>
+      </gazebo>
+      <gazebo reference="ur5_arm_gripper_left_tip">
+        <selfCollide>true</selfCollide>
+      </gazebo>
+      <gazebo reference="ur5_arm_gripper_right_tip">
         <selfCollide>true</selfCollide>
       </gazebo>

Commit message: - update the gripper URDF to the current actual gripper - update the gripper material to the black color

File: gripper/mybot_description/urdf/gripper.xacro (robot description, xacro)
@@ -3,15 +3,15 @@
 <link name='base'>
   <collision>
-    <origin xyz="0 0 0" rpy="0 0 0"/>
-    <geometry>
-      <mesh filename="package://mybot_description/meshes/base.DAE"/>
-    </geometry>
-  </collision>
-  <visual>
-  <origin xyz="0 0 0" rpy="0 0 0"/>
-    <geometry>
-<mesh filename="package://mybot_description/meshes/base.DAE"/>
-    </geometry>
-    <material name="white"/>
+    <origin xyz="0 -0.012 0" rpy="0 0 ${PI/2}"/>
+    <geometry>
+      <mesh filename="package://mybot_description/meshes/base_motor.DAE"/>
+    </geometry>
+  </collision>
+  <visual>
+  <origin xyz="0 -0.012 0" rpy="0 0 ${PI/2}"/>
+    <geometry>
+<mesh filename="package://mybot_description/meshes/base_motor.DAE"/>
+    </geometry>
+   <material name="black"/>
   </visual>
   <inertial>
@@ -24,5 +24,5 @@
   <parent link="base"/>
   <child link="link1"/>
- <origin xyz="0 0.005 -0.07" rpy="0 0 ${PI/2}"/>
+ <origin xyz="0 0 -0.07" rpy="0 0 ${PI/2}"/>
 </joint>
 <xacro:property name="PI" value="3.1415926535897931"/>
@@ -71,5 +71,5 @@
 <mesh filename="package://mybot_description/meshes/link1.DAE"/>
     </geometry>
-    <material name="white"/>
+   <material name="black"/>
   </visual>
   <inertial>
@@ -96,5 +96,5 @@
 <mesh filename="package://mybot_description/meshes/link2.DAE"/>
     </geometry>
-    <material name="white"/>
+   <material name="black"/>
   </visual>
   <inertial>
@@ -124,5 +124,5 @@
 <mesh filename="package://mybot_description/meshes/tip.DAE"/>
     </geometry>
-    <material name="white"/>
+   <material name="black"/>
   </visual>
   <inertial>
@@ -152,5 +152,5 @@
 <mesh filename="package://mybot_description/meshes/tip.DAE"/>
     </geometry>
-    <material name="white"/>
+   <material name="black"/>
   </visual>
   <inertial>

Commit message: Multiple Updates.

File: gripper/mybot_description/urdf/gripper.xacro (robot description, xacro)
@@ -3,13 +3,17 @@
 <link name='base'>
   <collision>
-    <origin xyz="0 -0.012 0" rpy="0 0 ${PI/2}"/>
-    <geometry>
-      <mesh filename="package://mybot_description/meshes/base_motor.DAE"/>
-    </geometry>
-  </collision>
-  <visual>
-  <origin xyz="0 -0.012 0" rpy="0 0 ${PI/2}"/>
-    <geometry>
-<mesh filename="package://mybot_description/meshes/base_motor.DAE"/>
+    <!-- origin xyz="0 -0.012 0" rpy="0 0 ${PI/2}"/ -->
+    <origin xyz="0 0 0" rpy="0 0 0"/>
+    <geometry>
+      <!-- mesh filename="package://mybot_description/meshes/base_motor.DAE"/ -->
+      <mesh filename="package://mybot_description/meshes/base.DAE"/>
+    </geometry>
+  </collision>
+  <visual>
+  <!-- origin xyz="0 -0.012 0" rpy="0 0 ${PI/2}"/ -->
+  <origin xyz="0 0 0" rpy="0 0 0"/>
+    <geometry>
+<!-- mesh filename="package://mybot_description/meshes/base_motor.DAE"/ -->
+<mesh filename="package://mybot_description/meshes/base.DAE"/>
     </geometry>
    <material name="black"/>
@@ -24,5 +28,6 @@
   <parent link="base"/>
   <child link="link1"/>
- <origin xyz="0 0 -0.07" rpy="0 0 ${PI/2}"/>
+ <!-- origin xyz="0 0 -0.07" rpy="0 0 ${PI/2}"/ -->
+ <origin xyz="0 0.005 -0.07" rpy="0 0 ${PI/2}"/>
 </joint>
 <xacro:property name="PI" value="3.1415926535897931"/>
@@ -109,5 +114,6 @@
 <origin xyz="0.0125 0 0.00025" rpy="0 0 -${PI/2}" />
   <axis xyz="0 0 1" rpy="0 0 0" />
-  <limit effort="100" velocity="5" lower="-0.037" upper="0.6" />
+  <!-- limit effort="100" velocity="5" lower="-0.037" upper="0.6" / -->
+  <limit effort="100" velocity="5" lower="-0.2" upper="0.6" />
   <joint_properties damping="0.0" friction="10.0"/>
 </joint>
@@ -137,5 +143,6 @@
 <origin xyz="-0.0125 0 0.00025" rpy="0 0 ${PI/2}" />
   <axis xyz="0 0 1" rpy="0 0 0" />
-  <limit effort="100" velocity="5" lower="-0.6" upper="0.037" />
+  <!-- limit effort="100" velocity="5" lower="-0.6" upper="0.037" / -->
+  <limit effort="100" velocity="5" lower="-0.6" upper="0.2" />
   <joint_properties damping="0.0" friction="10.0"/>
 </joint>
@@ -167,5 +174,5 @@
 <link name="camera">
   <collision>
-    <origin xyz="0 0 0" rpy="0 0 0"/>
+    <origin xyz="0.025 0 0" rpy="0 0 0"/>
     <geometry>
       <box size="${cameraSize*2} ${cameraSize/2} ${cameraSize/2}"/>
@@ -173,5 +180,5 @@
   </collision>
   <visual>
-   <origin xyz="0 0 0" rpy="0 0 0"/>
+   <origin xyz="0.025 0 0" rpy="0 0 0"/>
     <geometry>
       <box size="${cameraSize*2} ${cameraSize} ${cameraSize/2}"/>
@@ -181,5 +188,5 @@
   <inertial>
     <mass value="${cameraMass}" />
-    <origin xyz="0 0 0" rpy="0 0 0"/>
+    <origin xyz="0.025 0 0" rpy="0 0 0"/>
     <box_inertia m="${cameraMass}" x="${cameraSize*2}" y="${cameraSize}" z="${cameraSize/2}" />
   </inertial>

Commit message: fix the gripper grasping issue

File: gripper/mybot_description/urdf/gripper.xacro (robot description, xacro)
@@ -59,4 +59,6 @@
 <xacro:property name="tipWidth" value="0.03"/>
 <xacro:property name="tipMass" value="2.07"/>
+<xacro:property name="tip_close_limit" value="0.05"/>
+<xacro:property name="tip_open_limit" value="0.6"/>
 <xacro:property name="cameraSize" value="0.025"/>
 <xacro:property name="cameraMass" value="0.05"/>
@@ -112,8 +114,9 @@
   <parent link="link2"/>
   <child link="left_tip"/>
-<origin xyz="0.0125 0 0.00025" rpy="0 0 -${PI/2}" />
+<origin xyz="0.0125 0.001 0.0005" rpy="0 0 -${PI/2}" />
   <axis xyz="0 0 1" rpy="0 0 0" />
   <!-- limit effort="100" velocity="5" lower="-0.037" upper="0.6" / -->
-  <limit effort="100" velocity="5" lower="-0.2" upper="0.6" />
+  <!-- limit effort="100" velocity="5" lower="-0.2" upper="0.6" / -->
+  <limit effort="100" velocity="1" lower="${tip_close_limit}" upper="${tip_open_limit}" />
   <joint_properties damping="0.0" friction="10.0"/>
 </joint>
@@ -141,8 +144,9 @@
   <parent link="link2"/>
   <child link="right_tip"/>
-<origin xyz="-0.0125 0 0.00025" rpy="0 0 ${PI/2}" />
+<origin xyz="-0.0125 0.001 0.0005" rpy="0 0 ${PI/2}" />
   <axis xyz="0 0 1" rpy="0 0 0" />
   <!-- limit effort="100" velocity="5" lower="-0.6" upper="0.037" / -->
-  <limit effort="100" velocity="5" lower="-0.6" upper="0.2" />
+  <!-- limit effort="100" velocity="5" lower="-0.6" upper="0.2" / -->
+  <limit effort="100" velocity="1" lower="-${tip_open_limit}" upper="-${tip_close_limit}" />
   <joint_properties damping="0.0" friction="10.0"/>
 </joint>
@@ -212,3 +216,17 @@
   </actuator>
 </transmission>
+<!--adding the gripper tag-->
+<gazebo>
+  <gripper name="gripper">
+    <grasp_check>
+      <attach_steps>2</attach_steps>
+      <detach_steps>5000</detach_steps>
+      <min_contact_count>1</min_contact_count>
+    </grasp_check>
+    <!--gripper_link>right_tip</gripper_link-->
+    <!--gripper_link>left_tip</gripper_link-->
+    <gripper_link>link2</gripper_link>
+    <palm_link>link2</palm_link>
+  </gripper>
+</gazebo>
 </robot>

File: gripper/mybot_description/urdf/mybot.xacro (robot description, xacro)
@@ -16,17 +16,17 @@
 <xacro:property name="baseLength" value="0.01"/>
 <xacro:property name="baseWidth" value="0.08"/>
-<xacro:property name="baseMass" value="2.7"/>
+<xacro:property name="baseMass" value="0.6"/>
 <xacro:property name="link1Height" value="0.1"/>
 <xacro:property name="link1Length" value="0.2"/>
 <xacro:property name="link1Width" value="0.02"/>
-<xacro:property name="link1Mass" value="2.9"/>
+<xacro:property name="link1Mass" value="0.07"/>
 <xacro:property name="link2Height" value="0.12"/>
 <xacro:property name="link2Length" value="0.02"/>
 <xacro:property name="link2Width" value="0.02"/>
-<xacro:property name="link2Mass" value="2.2"/>
+<xacro:property name="link2Mass" value="0.01"/>
 <xacro:property name="tipHeight" value="0.3"/>
 <xacro:property name="tipLength" value="0.05"/>
 <xacro:property name="tipWidth" value="0.03"/>
-<xacro:property name="tipMass" value="2.07"/>
+<xacro:property name="tipMass" value="0.01"/>
 <xacro:property name="cameraSize" value="0.025"/>
 <xacro:property name="cameraMass" value="0.05"/>
@@ -164,7 +164,7 @@
   <parent link="link2"/>
   <child link="left_tip"/>
-<origin xyz="0.0125 0 0.00025" rpy="0 0 -${PI/2}" />
+<origin xyz="0.0125 0.001 0.0005" rpy="0 0 -${PI/2}" />
   <axis xyz="0 0 1" rpy="0 0 0" />
-  <limit effort="100" velocity="5" lower="-0.037" upper="0.6" />
+  <limit effort="100" velocity="1" lower="0.05" upper="0.6" />
   <joint_properties damping="0.0" friction="10.0"/>
 </joint>
@@ -192,7 +192,7 @@
   <parent link="link2"/>
   <child link="right_tip"/>
-<origin xyz="-0.0125 0 0.00025" rpy="0 0 ${PI/2}" />
+<origin xyz="-0.0125 0.001 0.0005" rpy="0 0 ${PI/2}" />
   <axis xyz="0 0 1" rpy="0 0 0" />
-  <limit effort="100" velocity="5" lower="-0.6" upper="0.037" />
+  <limit effort="100" velocity="1" lower="-0.6" upper="-0.05" />
   <joint_properties damping="0.0" friction="10.0"/>
 </joint>
@@ -262,3 +262,16 @@
   </actuator>
 </transmission>
+  <gazebo>
+    <gripper name="gripper">
+      <grasp_check>
+        <attach_steps>2</attach_steps>
+        <detach_steps>5000</detach_steps>
+        <min_contact_count>1</min_contact_count>
+      </grasp_check>
+      <!--gripper_link>right_tip</gripper_link-->
+      <!--gripper_link>left_tip</gripper_link-->
+      <gripper_link>link2</gripper_link>
+      <palm_link>link2</palm_link>
+    </gripper>
+  </gazebo>
 </robot>
