Commit message: Update to current

File: gripper/mybot_description/urdf/gripper.xacro (robot description, xacro)
@@ -3,13 +3,17 @@
 <link name='base'>
   <collision>
-    <origin xyz="0 -0.012 0" rpy="0 0 ${PI/2}"/>
-    <geometry>
-      <mesh filename="package://mybot_description/meshes/base_motor.DAE"/>
-    </geometry>
-  </collision>
-  <visual>
-  <origin xyz="0 -0.012 0" rpy="0 0 ${PI/2}"/>
-    <geometry>
-<mesh filename="package://mybot_description/meshes/base_motor.DAE"/>
+    <!-- origin xyz="0 -0.012 0" rpy="0 0 ${PI/2}"/ -->
+    <origin xyz="0 0 0" rpy="0 0 0"/>
+    <geometry>
+      <!-- mesh filename="package://mybot_description/meshes/base_motor.DAE"/ -->
+      <mesh filename="package://mybot_description/meshes/base.DAE"/>
+    </geometry>
+  </collision>
+  <visual>
+  <!-- origin xyz="0 -0.012 0" rpy="0 0 ${PI/2}"/ -->
+  <origin xyz="0 0 0" rpy="0 0 0"/>
+    <geometry>
+<!-- mesh filename="package://mybot_description/meshes/base_motor.DAE"/ -->
+<mesh filename="package://mybot_description/meshes/base.DAE"/>
     </geometry>
    <material name="black"/>
@@ -24,5 +28,6 @@
   <parent link="base"/>
   <child link="link1"/>
- <origin xyz="0 0 -0.07" rpy="0 0 ${PI/2}"/>
+ <!-- origin xyz="0 0 -0.07" rpy="0 0 ${PI/2}"/ -->
+ <origin xyz="0 0.005 -0.07" rpy="0 0 ${PI/2}"/>
 </joint>
 <xacro:property name="PI" value="3.1415926535897931"/>
@@ -54,4 +59,6 @@
 <xacro:property name="tipWidth" value="0.03"/>
 <xacro:property name="tipMass" value="2.07"/>
+<xacro:property name="tip_close_limit" value="0.05"/>
+<xacro:property name="tip_open_limit" value="0.6"/>
 <xacro:property name="cameraSize" value="0.025"/>
 <xacro:property name="cameraMass" value="0.05"/>
@@ -107,7 +114,9 @@
   <parent link="link2"/>
   <child link="left_tip"/>
-<origin xyz="0.0125 0 0.00025" rpy="0 0 -${PI/2}" />
+<origin xyz="0.0125 0.001 0.0005" rpy="0 0 -${PI/2}" />
   <axis xyz="0 0 1" rpy="0 0 0" />
-  <limit effort="100" velocity="5" lower="-0.037" upper="0.6" />
+  <!-- limit effort="100" velocity="5" lower="-0.037" upper="0.6" / -->
+  <!-- limit effort="100" velocity="5" lower="-0.2" upper="0.6" / -->
+  <limit effort="100" velocity="1" lower="${tip_close_limit}" upper="${tip_open_limit}" />
   <joint_properties damping="0.0" friction="10.0"/>
 </joint>
@@ -135,7 +144,9 @@
   <parent link="link2"/>
   <child link="right_tip"/>
-<origin xyz="-0.0125 0 0.00025" rpy="0 0 ${PI/2}" />
+<origin xyz="-0.0125 0.001 0.0005" rpy="0 0 ${PI/2}" />
   <axis xyz="0 0 1" rpy="0 0 0" />
-  <limit effort="100" velocity="5" lower="-0.6" upper="0.037" />
+  <!-- limit effort="100" velocity="5" lower="-0.6" upper="0.037" / -->
+  <!-- limit effort="100" velocity="5" lower="-0.6" upper="0.2" / -->
+  <limit effort="100" velocity="1" lower="-${tip_open_limit}" upper="-${tip_close_limit}" />
   <joint_properties damping="0.0" friction="10.0"/>
 </joint>
@@ -167,5 +178,5 @@
 <link name="camera">
   <collision>
-    <origin xyz="0 0 0" rpy="0 0 0"/>
+    <origin xyz="0.025 0 0" rpy="0 0 0"/>
     <geometry>
       <box size="${cameraSize*2} ${cameraSize/2} ${cameraSize/2}"/>
@@ -173,5 +184,5 @@
   </collision>
   <visual>
-   <origin xyz="0 0 0" rpy="0 0 0"/>
+   <origin xyz="0.025 0 0" rpy="0 0 0"/>
     <geometry>
       <box size="${cameraSize*2} ${cameraSize} ${cameraSize/2}"/>
@@ -181,5 +192,5 @@
   <inertial>
     <mass value="${cameraMass}" />
-    <origin xyz="0 0 0" rpy="0 0 0"/>
+    <origin xyz="0.025 0 0" rpy="0 0 0"/>
     <box_inertia m="${cameraMass}" x="${cameraSize*2}" y="${cameraSize}" z="${cameraSize/2}" />
   </inertial>
@@ -205,3 +216,17 @@
   </actuator>
 </transmission>
+<!--adding the gripper tag-->
+<gazebo>
+  <gripper name="gripper">
+    <grasp_check>
+      <attach_steps>2</attach_steps>
+      <detach_steps>5000</detach_steps>
+      <min_contact_count>1</min_contact_count>
+    </grasp_check>
+    <!--gripper_link>right_tip</gripper_link-->
+    <!--gripper_link>left_tip</gripper_link-->
+    <gripper_link>link2</gripper_link>
+    <palm_link>link2</palm_link>
+  </gripper>
+</gazebo>
 </robot>

Commit message: Fixed range estimate in idvalve.py and fixed spacing errors in rotate_valve.py

File: gripper/mybot_description/urdf/gripper.xacro (robot description, xacro)
@@ -60,5 +60,5 @@
 <xacro:property name="tipMass" value="2.07"/>
 <xacro:property name="tip_close_limit" value="0.05"/>
-<xacro:property name="tip_open_limit" value="0.6"/>
+<xacro:property name="tip_open_limit" value="1.0"/>
 <xacro:property name="cameraSize" value="0.025"/>
 <xacro:property name="cameraMass" value="0.05"/>

Commit message: First cut at using velodyne.

File: gripper/mybot_description/urdf/gripper.xacro (robot description, xacro)
@@ -1,5 +1,5 @@
 <?xml version="1.0"?>
 <robot name="mybot" xmlns:xacro="http://ros.org/wiki/xacro">
-<link name='base'>
+<link name='gripper_link'>
   <collision>
     <!-- origin xyz="0 -0.012 0" rpy="0 0 ${PI/2}"/ -->
@@ -26,5 +26,5 @@
 </link>
 <joint name="base_to_link1" type="fixed">
-  <parent link="base"/>
+  <parent link="gripper_link"/>
   <child link="link1"/>
  <!-- origin xyz="0 0 -0.07" rpy="0 0 ${PI/2}"/ -->
@@ -173,5 +173,5 @@
 <joint name="base_to_camera" type="fixed">
     <origin xyz="0 0 0" rpy="0 0 ${PI/2}"/>
-  <parent link="base"/>
+  <parent link="gripper_link"/>
   <child link="camera"/>
 </joint>

File: husky/husky_description/urdf/description.xacro (robot description, xacro)
@@ -22,4 +22,5 @@
 -->
 <robot name="husky" xmlns:xacro="http://ros.org/wiki/xacro">
+  <xacro:arg name="velodyne_lidar" default="false" />
   <xacro:arg name="laser_enabled" default="false" />
   <xacro:arg name="ur5_enabled" default="false" />

File: husky/husky_description/urdf/husky.urdf.xacro (robot description, xacro)
@@ -29,7 +29,9 @@
   <xacro:include filename="$(find husky_description)/urdf/accessories/primesense_carmine_1-09_camera.urdf.xacro"/>
   <xacro:include filename="$(find husky_description)/urdf/accessories/sick_lms1xx_mount.urdf.xacro"/>
+  <xacro:include filename="$(find husky_description)/urdf/accessories/velodyne_vlp16_mount.urdf.xacro"/>
   <xacro:include filename="$(find husky_description)/urdf/accessories/sensor_arch.urdf.xacro"/>
   <xacro:include filename="$(find ur_description)/urdf/ur5.urdf.xacro" />
   <xacro:include filename="$(find mybot_description)/urdf/gripper.xacro" />
+  <xacro:include filename="$(find velodyne_description)/urdf/VLP-16.urdf.xacro" />
   <property name="M_PI" value="3.14159"/>
   <!-- Base Size -->
@@ -128,5 +130,5 @@
         <joint name="base_to_arm" type="fixed">
           <parent link="ur5_arm_wrist_3_link"/>
-          <child link="base"/>
+          <child link="gripper_link"/>
           <origin xyz="0 0.09 0" rpy="0 0 0"/>
         </joint>
@@ -143,5 +145,5 @@
       </joint>
     </xacro:if>
-    <!-- Spawn LIDAR if laser_enabled = "true" -->
+    <!-- Spawn sick_lms1xx -->
     <xacro:if value="$(arg laser_enabled)">
       <sick_lms1xx_mount prefix="base" topic="scan"/>
@@ -152,4 +154,17 @@
         <child link="base_laser_mount" />
       </joint>
+    </xacro:if>
+    <!-- Spawn velodyne vlp-16 -->
+    <xacro:if value="$(arg velodyne_lidar)">
+      <VLP-16 parent="top_plate_link" name="laser" topic="velodyne_points" >
+        <origin xyz="0.415 0 -0.08" rpy="0 0 0" />
+      </VLP-16>
+      <!-- velodyne_vlp16_mount prefix="base" topic="velodyne_points"/ -->
+      <!-- joint name="laser_mount_joint" type="fixed">
+        <origin xyz="$(optenv HUSKY_LMS1XX_XYZ 0.415 0.0 -0.04)"
+                rpy="$(optenv HUSKY_LMS1XX_RPY 0.0 0.0 0.0)" />
+        <parent link="top_plate_link" />
+        <child link="base_laser_mount" />
+      </joint -->
     </xacro:if>
     <!-- Spawn Kinect if kinect_enabled = "true" -->

File: husky/husky_simulator/husky_gazebo/urdf/description.gazebo.xacro (robot description, xacro)
@@ -23,4 +23,5 @@
 <robot name="husky" xmlns:xacro="http://ros.org/wiki/xacro">
 <!-- <robot name="husky_robot_gazebo" xmlns:xacro="http://ros.org/wiki/xacro"> -->
+  <xacro:arg name="velodyne_lidar" default="false"/>
   <xacro:arg name="laser_enabled" default="true" />
   <xacro:arg name="ur5_enabled" default="false" />
