Commit message: Updating VTREX packages.

File: vtrex_description/urdf/macros.xacro (robot description, xacro)
@@ -2,21 +2,21 @@
 <robot name="vtrex" xmlns:xacro="http://www.ros.org/wiki/xacro">
   <xacro:property name="PI" value="3.1415926535897931" />
-  <xacro:property name="wheelbase" value="0.262" />
-  <xacro:property name="track" value="0.37559" />
-  <xacro:property name="wheel_vertical_offset" value="0.0345" />
-  <xacro:property name="footprint_vertical_offset" value="-0.0655" />
-  <xacro:property name="wheel_radius" value="0.098" />
-  <xacro:property name="wheel_width" value="0.040" />
-  <xacro:property name="chassis_length" value="0.420" />
-  <xacro:property name="chassis_width" value="0.310" />
-  <xacro:property name="chassis_height" value="0.184" />
+ <xacro:property name="wheelbase" value="0.7" />
+  <xacro:property name="track" value="0.64" />
+  <xacro:property name="wheel_vertical_offset" value="0.1651" />
+  <xacro:property name="footprint_vertical_offset" value=".24866" />
+  <xacro:property name="wheel_radius" value="0.1651" />
+  <xacro:property name="wheel_width" value="0.1016" />
+  <xacro:property name="chassis_length" value="0.95" />
+  <xacro:property name="chassis_width" value="0.747" />
+  <xacro:property name="chassis_height" value="0.41" />
   <xacro:property name="dummy_inertia" value="1e-09"/>
   <xacro:property name="mount_spacing" value="0.120" />
-<macro name="wheel" params="prefix *joint_pose">
+<xacro:macro name="wheel" params="prefix *joint_pose">
     <link name="${prefix}_wheel_link">
       <visual>
-        <origin xyz="0 0 0" rpy="${PI/2} 0 0"/>
+        <origin xyz="0 0 0" rpy="0 0 0"/>
         <geometry>
-          <mesh filename="package://vtrex_description/meshes/wheel.STL"/>
+       <mesh filename="package://vtrex_description/meshes/wheel.STL"/>
         </geometry>
         <material name="black" />
@@ -25,14 +25,14 @@
         <origin xyz="0 0 0" rpy="${PI/2} 0 0"/>
         <geometry>
-          <cylinder radius="${wheel_radius}" length="${wheel_width}"/>
+         <cylinder radius="${wheel_radius}" length="${wheel_width}"/>
         </geometry>
       </collision>
       <inertial>
         <origin xyz="0 0 0" rpy="0 0 0"/>
-        <mass value="0.477"/>
+        <mass value="4.25"/>
         <inertia
-          ixx="0.0013" ixy="0" ixz="0"
-          iyy="0.0024" iyz="0"
-          izz="0.0013"/>
+          ixx="0.03" ixy="0" ixz="0"
+          iyy="0.263" iyz="0"
+          izz="0.03"/>
       </inertial>
     </link>

File: vtrex_description/urdf/vtrex.xacro (robot description, xacro)
@@ -1,9 +1,5 @@
 <?xml version="1.0"?>
 <robot name="vtrex" xmlns:xacro="http://www.ros.org/wiki/xacro">
-  <xacro:arg name="velodyne_lidar" default="true"/>
-  <xacro:arg name="laser_enabled" default="false" />
-  <xacro:arg name="ur5_enabled" default="true" />
-  <xacro:arg name="ur5_camera_enabled" default="false" />
-  <xacro:property name="M_PI" value="3.1415926535897931" />
+  <xacro:property name="PI" value="3.1415926535897931" />
   <xacro:property name="wheelbase" value="0.7" />
   <xacro:property name="track" value="0.64" />
@@ -15,16 +11,16 @@
   <xacro:property name="wheel_width" value="0.1016" />
   <xacro:property name="chassis_length" value="0.95" />
-  <xacro:property name="chassis_width" value="0.48" />
-  <xacro:property name="chassis_height" value="0.28" />
+  <xacro:property name="chassis_width" value="0.747" />
+  <xacro:property name="chassis_height" value="0.41" />
   <xacro:property name="dummy_inertia" value="1e-09"/>
   <xacro:property name="cameraSize" value="0.025"/>
   <xacro:property name="cameraMass" value="0.05"/>
   <xacro:include filename="$(find vtrex_description)/urdf/vtrex.gazebo" />
-  <xacro:include filename="$(find vtrex_description)/urdf/accessories/sick_lms1xx_mount.urdf.xacro"/>
-  <xacro:include filename="$(find husky_description)/urdf/accessories/velodyne_vlp16_mount.urdf.xacro"/>
-  <xacro:include filename="$(find ur_description)/urdf/ur5.urdf.xacro" />
-  <xacro:include filename="$(find mybot_description)/urdf/gripper.xacro" />
-  <xacro:include filename="$(find velodyne_description)/urdf/VLP-16.urdf.xacro" />
-  <xacro:macro name="wheel" params="prefix *joint_pose">
+  <xacro:include filename="$(find vtrex_description)/urdf/materials.xacro" />
+  <xacro:include filename="$(find velodyne_description)/urdf/HDL-32E.urdf.xacro" />
+<!--############################################sicklms1xx#################################################
+<xacro:include filename="$(find LMS1xx)/urdf/sick_lms1xx.urdf.xacro" />
+-->
+<xacro:macro name="wheel" params="prefix *joint_pose">
     <link name="${prefix}_wheel_link">
       <visual>
@@ -36,5 +32,5 @@
       </visual>
       <collision>
-        <origin xyz="0 0 0" rpy="${M_PI/2} 0 0"/>
+        <origin xyz="0 0 0" rpy="${PI/2} 0 0"/>
         <geometry>
          <cylinder radius="${wheel_radius}" length="${wheel_width}"/>
@@ -43,8 +39,8 @@
       <inertial>
         <origin xyz="0 0 0" rpy="0 0 0"/>
-        <mass value="3.4"/>
+        <mass value="4.25"/>
         <inertia
           ixx="0.03" ixy="0" ixz="0"
-          iyy="0.05" iyz="0"
+          iyy="0.263" iyz="0"
           izz="0.03"/>
       </inertial>
@@ -107,10 +103,10 @@
       <origin xyz="0.00  0.00 ${footprint_vertical_offset}" rpy="0 0 0"/>
        <!--<origin xyz="0.012  0.002 0.067" rpy="0 0 0"/>-->
-      <mass value="40"/>
+      <mass value="35"/>
       <!-- Moments of inertia: ( chassis without wheels ) -->
       <inertia
-        ixx="2" ixy="-0.01" ixz="-0.00"
+        ixx="2" ixy="-0.00" ixz="-0.00"
         iyy="3.68" iyz="-0.0000"
-        izz="4.85"/>
+        izz="5.42"/>
       </inertial>
   </link>
@@ -177,53 +173,23 @@
     </joint>
     <joint name="right_wheel_cover" type="fixed">
-      <origin xyz="0 0 0" rpy="0 0 ${M_PI}" />
+      <origin xyz="0 0 0" rpy="0 0 ${PI}" />
       <parent link="chassis_link"/>
       <child link="right_wheel_cover_link" />
     </joint>
 <!--############################################wheelscover#################################################-->
-    <link name="imu_link">
-      <inertial>
-        <mass value="0.001"/>
-        <origin xyz="0 0 0" rpy="0 0 0"/>
-        <inertia ixx="${dummy_inertia}" ixy="0.0" ixz="0.0" iyy="${dummy_inertia}" iyz="0.0" izz="${dummy_inertia}"/>
-      </inertial>
-    </link>
-    <joint name="imu_joint" type="fixed">
-      <parent link="chassis_link" />
-      <child link="imu_link" />
-    </joint>
-    <xacro:if value="$(arg laser_enabled)">
-      <sick_lms1xx_mount prefix="base" topic="scan"/>
-      <joint name="laser_mount_joint" type="fixed">
-        <origin xyz="$(optenv vtrex_LMS1XX_XYZ 0.5206 0.0 0.1135)"
-                rpy="$(optenv vtrex_LMS1XX_RPY 0.0 0.0 0.0)" />
-        <parent link="chassis_link" />
-        <child link="base_laser_mount" />
-      </joint>
-    </xacro:if>
-    <xacro:if value="$(arg ur5_enabled)">
-      <xacro:property name="reflect" value="-1" />
-      <!-- Spawn arm -->
-      <xacro:ur5_robot prefix="ur5_arm_" joint_limited="true"/>
-      <!-- Join arm -->
-      <joint name="ur5_arm_base" type="fixed">
-        <parent link="chassis_link" />
-        <child link="ur5_arm_base_link" />
-        <origin xyz="0.3058 0 0.375" rpy="0.0 0.0 -1.57079632679" />
-      </joint>
-      <!--Spawn gripper-->
-      <xacro:gripper />
-      <!-- Join Gripper -->
-        <joint name="base_to_arm" type="fixed">
-          <parent link="ur5_arm_wrist_3_link"/>
-          <child link="gripper_link"/>
-          <origin xyz="0 0.09 0" rpy="0 0 0"/>
-        </joint>
-    </xacro:if>
-    <!-- Spawn velodyne vlp-16 -->
-    <xacro:if value="$(arg velodyne_lidar)">
-      <VLP-16 parent="chassis_link" name="laser" topic="velodyne_points" >
-        <origin xyz="0.5206 0.0 0.1135" rpy="0 0 0" />
-      </VLP-16>
-    </xacro:if>
+  <link name="imu_link">
+    <inertial>
+      <mass value="0.001"/>
+      <origin xyz="0 0 0" rpy="0 0 0"/>
+      <inertia ixx="${dummy_inertia}" ixy="0.0" ixz="0.0" iyy="${dummy_inertia}" iyz="0.0" izz="${dummy_inertia}"/>
+    </inertial>
+  </link>
+  <joint name="imu_joint" type="fixed">
+    <parent link="chassis_link" />
+    <child link="imu_link" />
+  </joint>
+<!--############################################VELODYNE##################################################-->
+    <HDL-32E parent="base_link" name="velodyne_link" topic="velodyne_points" >
+      <origin xyz="0.6 0 0.23" rpy="0 0 -1.57"/>
+    </HDL-32E>
 </robot>

Commit message: Updated some of vtrex urdf to work with sawyer.

File: vtrex_description/urdf/macros.xacro (robot description, xacro)
@@ -20,5 +20,5 @@
        <mesh filename="package://vtrex_description/meshes/wheel.STL"/>
         </geometry>
-        <material name="black" />
+        <material name="vtrex_black" />
       </visual>
       <collision>

File: vtrex_description/urdf/materials.xacro (robot description, xacro)
@@ -1,12 +1,12 @@
 <?xml version="1.0"?>
 <robot name="vtrex" xmlns:xacro="http://www.ros.org/wiki/xacro">
-<material name="blue"><color rgba="0.0 0.0 0.8 1.0"/></material>
-<material name="green"><color rgba="0.0 0.8 0.0 1.0"/></material>
-<material name="grey"><color rgba="0.2 0.2 0.2 1.0"/></material>
-<material name="orange"><color rgba="${255/255} ${108/255} ${10/255} 1.0"/></material>
-<material name="red"><color rgba="0.8 0.0 0.0 1.0"/></material>
-<material name="white"><color rgba="1.0 1.0 1.0 1.0"/></material>
-<material name="dark_grey"><color rgba="0.2 0.2 0.2 1.0" /></material>
-<material name="light_grey"><color rgba="0.4 0.4 0.4 1.0" /></material>
-<material name="black"><color rgba="0.15 0.15 0.15 1.0" /></material>
+<material name="vtrex_blue"><color rgba="0.0 0.0 0.8 1.0"/></material >
+<material name="vtrex_green"><color rgba="0.0 0.8 0.0 1.0"/></material >
+<material name="vtrex_grey"><color rgba="0.2 0.2 0.2 1.0"/></material >
+<material name="vtrex_orange"><color rgba="${255/255} ${108/255} ${10/255} 1.0"/></material>
+<material name="vtrex_red"><color rgba="0.8 0.0 0.0 1.0"/></material>
+<material name="vtrex_white"><color rgba="1.0 1.0 1.0 1.0"/></material>
+<material name="vtrex_dark_grey"><color rgba="0.2 0.2 0.2 1.0" /></material>
+<material name="vtrex_light_grey"><color rgba="0.4 0.4 0.4 1.0" /></material>
+<material name="vtrex_black"><color rgba="0.15 0.15 0.15 1.0" /></material>
 </robot>

File: vtrex_description/urdf/vtrex.xacro (robot description, xacro)
@@ -1,4 +1,5 @@
 <?xml version="1.0"?>
 <robot name="vtrex" xmlns:xacro="http://www.ros.org/wiki/xacro">
+  <xacro:arg name="sawyer_enabled" default="true" />
   <xacro:property name="PI" value="3.1415926535897931" />
   <xacro:property name="wheelbase" value="0.7" />
@@ -19,4 +20,6 @@
   <xacro:include filename="$(find vtrex_description)/urdf/materials.xacro" />
   <xacro:include filename="$(find velodyne_description)/urdf/HDL-32E.urdf.xacro" />
+  <xacro:include filename="$(find sawyer_description)/urdf/sawyer.urdf" />
+  <xacro:include filename="$(find mybot_description)/urdf/gripper.xacro" />
 <!--############################################sicklms1xx#################################################
 <xacro:include filename="$(find LMS1xx)/urdf/sick_lms1xx.urdf.xacro" />
@@ -29,5 +32,5 @@
        <mesh filename="package://vtrex_description/meshes/wheel.STL"/>
         </geometry>
-        <material name="black" />
+        <material name="vtrex_black" />
       </visual>
       <collision>
@@ -91,5 +94,5 @@
        <mesh filename="package://vtrex_description/meshes/Chassis.STL"/>
       </geometry>
-<material name="black" />
+<material name="vtrex_black" />
      </visual>
     <collision>
@@ -121,5 +124,5 @@
        <mesh filename="package://vtrex_description/meshes/wheelscover.STL"/>
         </geometry>
-        <material name="red" />
+        <material name="vtrex_red" />
       </visual>
       <collision>
@@ -144,5 +147,5 @@
        <mesh filename="package://vtrex_description/meshes/wheelscover.STL"/>
         </geometry>
-        <material name="red" />
+        <material name="vtrex_red" />
       </visual>
       <collision>
@@ -193,3 +196,21 @@
       <origin xyz="0.6 0 0.23" rpy="0 0 -1.57"/>
     </HDL-32E>
+<!--############################################SAWYER##################################################-->
+    <xacro:if value="$(arg sawyer_enabled)">
+      <xacro:property name="reflect" value="-1" />
+      <!-- Spawn arm -->
+      <joint name="sawyer_arm_base" type="fixed">
+        <parent link="chassis_link" />
+        <child link="base" />
+        <origin xyz="0.3058 0 0.375" rpy="0.0 0.0 0" />
+      </joint>
+      <!--Spawn gripper-->
+      <xacro:gripper />
+      <!-- Join Gripper -->
+        <joint name="base_to_arm" type="fixed">
+          <parent link="right_l6"/>
+          <child link="gripper_link"/>
+          <origin xyz="0.0 0.0 0.05" rpy="1.57 0 1.57"/>
+        </joint>
+    </xacro:if>
 </robot>
