Commit message: Updates from physical VTREX.

File: gripper/gripper_description/urdf/gripper.urdf.xacro (robot description, xacro)
@@ -62,5 +62,5 @@
 	     </link>
 	     <joint name="${prefix}base_link_link_1_joint" type="fixed">
-	       <parent link="${prefix}base_link"/>
+	       <parent link="gripper_link"/>
 	       <child link="${prefix}link_1"/>
 	       <origin xyz="0 0.005 -0.07" rpy="0 0 ${PI/2}"/>
@@ -165,5 +165,5 @@
 	    <joint name="${prefix}base_link_camera_joint" type="fixed">
 	      <origin xyz="0 0 0" rpy="0 0 0"/>
-	      <parent link="${prefix}base_link"/>
+	      <parent link="gripper_link"/>
 	      <child link="${prefix}camera_link"/>
 	    </joint>

File: vtrex_description/urdf/vtrex.xacro (robot description, xacro)
@@ -1,5 +1,7 @@
 <?xml version="1.0"?>
 <robot name="vtrex" xmlns:xacro="http://www.ros.org/wiki/xacro">
-  <xacro:arg name="sawyer_enabled" default="true" />
+  <xacro:arg name="sawyer_enabled" default="false" />
+  <xacro:arg name="ur5_enabled" default="true" />
+  <xacro:arg name="velodyne_enabled" default="true" />
   <xacro:property name="PI" value="3.1415926535897931" />
   <xacro:property name="wheelbase" value="0.7" />
@@ -19,6 +21,8 @@
   <xacro:include filename="$(find vtrex_description)/urdf/vtrex.gazebo" />
   <xacro:include filename="$(find vtrex_description)/urdf/materials.xacro" />
+  <xacro:include filename="$(find vtrex_description)/urdf/microstrain.xacro" />
   <xacro:include filename="$(find velodyne_description)/urdf/HDL-32E.urdf.xacro" />
-  <xacro:include filename="$(find sawyer_description)/urdf/sawyer.urdf" />
+  <xacro:include filename="$(find ur_description)/urdf/ur5.urdf.xacro" />
+  <!--xacro:include filename="$(find sawyer_description)/urdf/sawyer.urdf" / -->
   <xacro:include filename="$(find mybot_description)/urdf/gripper.xacro" />
 <!--############################################sicklms1xx#################################################
@@ -181,5 +185,7 @@
     </joint>
 <!--############################################wheelscover#################################################-->
-  <link name="imu_link">
+<!--############################################IMU####################################################-->
+<!--xacro:microstrain_sensor sensorName="mstrain" parentLink="imu_link" origin_xyz="0 0 0" origin_rpy="0 0 0"/ -->
+  <link name="imu">
     <inertial>
       <mass value="0.001"/>
@@ -190,10 +196,30 @@
   <joint name="imu_joint" type="fixed">
     <parent link="chassis_link" />
-    <child link="imu_link" />
+    <origin xyz="-0.145 0.000 0.15" rpy="0 0 0" />
+    <child link="imu" />
   </joint>
 <!--############################################VELODYNE##################################################-->
-    <HDL-32E parent="base_link" name="velodyne_link" topic="velodyne_points" >
-      <origin xyz="0.6 0 0.23" rpy="0 0 -1.57"/>
-    </HDL-32E>
+      <HDL-32E parent="base_link" name="velodyne_link" topic="velodyne_points" >
+        <origin xyz="0.6 0 0.23" rpy="0 0 -1.57"/>
+      </HDL-32E>
+<!--############################################UR5##################################################-->
+    <xacro:if value="$(arg ur5_enabled)">
+      <xacro:property name="reflect" value="-1" />
+      <!-- Spawn arm -->
+      <xacro:ur5_robot prefix="ur5_arm_" joint_limited="true"/>
+      <!-- Join arm -->
+      <joint name="ur5_arm_base" type="fixed">
+        <parent link="chassis_link" />
+        <child link="ur5_arm_base_link" />
+        <origin xyz="0.335 0 0.375" rpy="0.0 0.0 -1.57079632679" />
+      </joint>
+      <!--Spawn gripper-->
+      <xacro:gripper />
+        <joint name="base_to_arm" type="fixed">
+          <parent link="ur5_arm_wrist_3_link"/>
+          <child link="gripper_link"/>
+          <origin xyz="0.0 0.0823 0.0" rpy="0 0 0"/>
+        </joint>
+    </xacro:if>
 <!--############################################SAWYER##################################################-->
     <xacro:if value="$(arg sawyer_enabled)">

Commit message: Update gripper mass.

File: gripper/gripper_description/urdf/gripper.urdf.xacro (robot description, xacro)
@@ -10,19 +10,19 @@
   <xacro:property name="baseLength" value="0.01"/>
   <xacro:property name="baseWidth" value="0.08"/>
-  <xacro:property name="baseMass" value="2.7"/>
+  <xacro:property name="baseMass" value="0.0001"/>
   <xacro:property name="link1Height" value="0.1"/>
   <xacro:property name="link1Length" value="0.2"/>
   <xacro:property name="link1Width" value="0.02"/>
-  <xacro:property name="link1Mass" value="2.9"/>
+  <xacro:property name="link1Mass" value="0.0001"/>
   <xacro:property name="link2Height" value="0.12"/>
   <xacro:property name="link2Length" value="0.02"/>
   <xacro:property name="link2Width" value="0.02"/>
-  <xacro:property name="link2Mass" value="2.2"/>
+  <xacro:property name="link2Mass" value="0.0001"/>
   <xacro:property name="tipHeight" value="0.3"/>
   <xacro:property name="tipLength" value="0.05"/>
   <xacro:property name="tipWidth" value="0.03"/>
-  <xacro:property name="tipMass" value="2.07"/>
+  <xacro:property name="tipMass" value="0.0001"/>
   <xacro:property name="cameraSize" value="0.025"/>
-  <xacro:property name="cameraMass" value="0.05"/>
+  <xacro:property name="cameraMass" value="0.0001"/>
   <xacro:property name="chassisHeight" value="0.05"/>
   <xacro:property name="chassisLength" value="0.15"/>
